File: pcb/pcb.kicad_pcb (KiCad board)
At the start: 2 copper layers, 111 parts, among them U0 Teensy4.1

Commit message: Ok
Parts:
- moved REF9 323.7 mm to (69.5, 71.3)
- moved REF38 320.5 mm to (79.5, 123.3)
- moved REF10 319.3 mm to (89.5, 71.3)
- moved REF8 314.8 mm to (49.5, 71.3)
- moved REF4 308.6 mm to (99.5, 54.0)
- moved REF22 299.3 mm to (79.5, 88.6)
- moved REF42 287.8 mm to (109.5, 140.6)
- moved REF40 283.3 mm to (69.5, 140.6)
- moved REF41 272.1 mm to (89.5, 140.6)
- moved REF35 241.0 mm to (139.5, 123.3)
- moved REF12 234.5 mm to (129.5, 71.3)
- moved REF18 221.2 mm to (159.5, 88.6)
- moved REF21 219.5 mm to (99.5, 88.6)
- moved REF37 214.9 mm to (99.5, 123.3)
- moved REF23 214.5 mm to (59.5, 88.6)
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- renumbered REF0 to REF1, REF0 to REF10, REF0 to REF11, REF0 to REF12, REF0 to REF13, REF0 to REF14, REF0 to REF15, REF0 to REF16, REF0 to REF17, REF0 to REF18, REF0 to REF19, REF0 to REF2, REF0 to REF20, REF0 to REF21, REF0 to REF22, REF0 to REF23, REF0 to REF24, REF0 to REF25, REF0 to REF26, REF0 to REF27, REF0 to REF28, REF0 to REF29, REF0 to REF3, REF0 to REF30, REF0 to REF31, REF0 to REF32, REF0 to REF33, REF0 to REF34, REF0 to REF35, REF0 to REF36, REF0 to REF37, REF0 to REF38, REF0 to REF39, REF0 to REF4, REF0 to REF40, REF0 to REF41, REF0 to REF42, REF0 to REF43, REF0 to REF44, REF0 to REF45, REF0 to REF46, REF0 to REF47, REF0 to REF5, REF0 to REF6, REF0 to REF7, REF0 to REF8, REF0 to REF9
Routing:
- net CONTROL0: track 0.00 -> 162.7 mm, vias 0 -> 3
- net CONTROL1: track 0.00 -> 160.1 mm, vias 0 -> 3
- net CONTROL2: track 0.00 -> 156.8 mm, vias 0 -> 3
- net CONTROL3: track 0.00 -> 154.2 mm, vias 0 -> 3
- net AM2: track 0.00 -> 103.1 mm, vias 0 -> 1
- net AM1:8: track 0.00 -> 79.4 mm
- net AM0:7: track 0.00 -> 78.7 mm
- net AM2:7: track 0.00 -> 77.9 mm
- net AM2:15: track 0.00 -> 73.1 mm
- net AM0:15: track 0.00 -> 72.7 mm
- net AM1:0: track 0.00 -> 71.7 mm
- net AM1:7: track 0.00 -> 69.0 mm
- net AM0:8: track 0.00 -> 69.0 mm
- net AM2:8: track 0.00 -> 68.2 mm
- net AM1: track 0.00 -> 65.2 mm, vias 0 -> 1
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- added copper zone on B.Cu, net +3.3V
- added copper zone on F.Cu, net GND
Other:
- board outline added: 207 x 133 mm
