File: pcb/pcb.kicad_sch (KiCad schematic)
At the start: 63 parts, among them U0 Teensy4.1

Commit message: Feedback
Parts:
- added C0, C1, C10, C2, C3, C4, C5, C6, C7, C8, C9: 100nF, symbol Device:C
Connections:
- net +3.3V: now also C0.1, C1.1, C10.2, C2.1, C3.2, C4.2, C5.2, C6.2, C7.2, C8.2, C9.2
- net GND: now also C0.2, C1.2, C10.1, C2.2, C3.1, C4.1, C5.1, C6.1, C7.1, C8.1, C9.1
Other:
- moved on the sheet: AM0, AM1, AM2, FID1, FID2, FID3, H1, H2, H3, H4, H5, H6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

Commit message: Feedback
Parts:
- added C11, C12: 10u, Capacitor_SMD:C_0402_1005Metric, symbol Device:C_Small
- added J1: Barrel_Jack, symbol Connector:Barrel_Jack
- added LDO1: AMS1117-3.3, Package_TO_SOT_SMD:SOT-223-3_TabPin2, symbol Regulator_Linear:AMS1117-3.3
Connections:
- net +3.3V: now also C12.1, LDO1.2 (VO); no longer U0.51 (3V3)
- net GND: now also U0.1 (GND), U0.34 (GND), U0.47 (GND), U0.58 (GND), U0.59 (GND), U0.64 (GND), C11.2, C12.2, J1.2, LDO1.1 (GND)
- new net +5V: C11.1, J1.1, LDO1.3 (VI)
Other:
- note added: "External power input (powers everything except Teensy)"
- moved on the sheet: AM0, AM1, AM2, C0, C1, C10, C2, C3, C4, C5, C6, C7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

Commit message: Ok
Parts:
- C0, C1, C10, C2, C3, C4, C5, C6, C7, C8, C9: footprint (none) -> Capacitor_SMD:C_0402_1005Metric
