File: kicad/3_key/3_key.kicad_pcb (KiCad board)
At the start: 2 copper layers, 85 x 75 mm, 25 parts, among them J1 EJ508A, U1 Teensy4.1

Commit message: Ok
Parts:
- removed H5: MountingHole, MountingHole:MountingHole_3.2mm_M3_Pad
- removed J1: EJ508A, EJ508A:MPD_EJ508A
- added DC0: DC-005-A250, easyeda2kicad:DC-IN-TH_DC-005-A250, F.Cu at (42.8, 63.1)
- added U2: X6511FV-24-C85D32, easyeda2kicad:HDR-TH_24P-P2.54-V-F, F.Cu at (64.5, 31.8)
- AM0: value CD74HC4067SM -> CD74HC4067SM96; footprint Package_SO:SSOP-24_5.3x8.2mm_P0.65mm -> easyeda2kicad:SSOP-24_L8.1-W5.3-P0.65-LS7.8-BL; moved to F.Cu
- C0, C1, C2, C3: value 100nF -> CL05B104KA5NNNC; footprint GCM155R71C104KA55D:CAPC1005X55N -> easyeda2kicad:C0402; moved to F.Cu
- C4, C5: value 10uF -> CL10A106MQ8NNNC; footprint GRM21BC81A106KE18L:CAPC2012X135N -> easyeda2kicad:C0603; moved to F.Cu
- LDO1: value AMS1117-3.3 -> AMS1085CM-3.3; footprint Package_TO_SOT_SMD:SOT-223-3_TabPin2 -> easyeda2kicad:TO-263-3_L8.6-W10.2-P2.54-LS14.4-TL; moved to F.Cu
- R0: value 1k ohm -> 1206W4F1001T5E; footprint RC0603JR-071KL:RESC1607X60N -> easyeda2kicad:R1206; moved to F.Cu
- REF0, REF1, REF2: moved to B.Cu
- S0, S1, S2: value Hall_Sensor -> GH39FKSW; footprint Package_TO_SOT_SMD:SOT-23 -> easyeda2kicad:SOT-23-3_L2.9-W1.3-P1.90-LS2.4-BR; moved to F.Cu
- U1: value Teensy4.1 -> X6511FV-24-C85D32; footprint teensy:Teensy41 -> easyeda2kicad:HDR-TH_24P-P2.54-V-F
- moved H4 173.0 mm to (82.0, 68.6)
- moved C1 158.9 mm to (82.0, 54.5), turned to 0 degrees
- moved REF1 158.6 mm to (82.0, 58.3), turned to 180 degrees
- moved S1 158.6 mm to (82.0, 58.3), turned to 0 degrees
- moved AM0 157.5 mm to (53.5, 77.0), turned to 0 degrees
- moved C3 155.2 mm to (50.0, 71.1)
- moved H2 153.5 mm to (97.7, 25.7)
- moved FID2 150.6 mm to (91.1, 52.1)
- moved C4 149.8 mm to (52.3, 63.3), turned to -90 degrees
- moved H3 147.9 mm to (30.4, 79.0)
- moved FID1 147.4 mm to (28.9, 35.1)
- moved U1 147.4 mm to (64.5, 47.0)
- moved R0 146.6 mm to (74.9, 28.4), turned to 0 degrees
- moved H1 145.9 mm to (30.4, 25.7)
- moved C0 145.4 mm to (71.8, 72.1), turned to 0 degrees
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Connections:
- C3 pad 1: GND -> +3.3V
- C3 pad 2: +3.3V -> GND
- C4 pad 1: GND -> +5V
- C4 pad 2: +3.3V -> GND
- C5 pad 1: GND -> +3.3V
- C5 pad 2: +5V -> GND
- R0 pad 1: Net-(U1-41_A17) -> Net-(U0-41_A17)
- U1 pad 10: unconnected-(U1-8_TX2_IN1-Pad10) -> Net-(U0-8_TX2_IN1)
- U1 pad 11: unconnected-(U1-9_OUT1C-Pad11) -> Net-(U0-9_OUT1C)
- U1 pad 12: unconnected-(U1-10_CS_MQSR-Pad12) -> Net-(U0-10_CS_MQSR)
- U1 pad 13: unconnected-(U1-11_MOSI_CTX1-Pad13) -> Net-(U0-11_MOSI_CTX1)
- U1 pad 14: unconnected-(U1-12_MISO_MQSL-Pad14) -> Net-(U0-12_MISO_MQSL)
- U1 pad 15: unconnected-(U1-3V3-Pad15) -> Net-(U0-3V3-Pad15)
- U1 pad 16: unconnected-(U1-24_A10_TX6_SCL2-Pad16) -> Net-(U0-24_A10_TX6_SCL2)
- U1 pad 17: unconnected-(U1-25_A11_RX6_SDA2-Pad17) -> Net-(U0-25_A11_RX6_SDA2)
- U1 pad 18: unconnected-(U1-26_A12_MOSI1-Pad18) -> Net-(U0-26_A12_MOSI1)
- U1 pad 19: unconnected-(U1-27_A13_SCK1-Pad19) -> Net-(U0-27_A13_SCK1)
- U1 pad 2: unconnected-(U1-0_RX1_CRX2_CS1-Pad2) -> Net-(U0-0_RX1_CRX2_CS1)
- U1 pad 20: unconnected-(U1-28_RX7-Pad20) -> Net-(U0-28_RX7)
- U1 pad 21: unconnected-(U1-29_TX7-Pad21) -> Net-(U0-29_TX7)
- U1 pad 22: unconnected-(U1-30_CRX3-Pad22) -> Net-(U0-30_CRX3)
- U1 pad 23: unconnected-(U1-31_CTX3-Pad23) -> Net-(U0-31_CTX3)
- U1 pad 24: unconnected-(U1-32_OUT1B-Pad24) -> Net-(U0-32_OUT1B)
- U1 pad 3: unconnected-(U1-1_TX1_CTX2_MISO1-Pad3) -> Net-(U0-1_TX1_CTX2_MISO1)
- U1 pad 8: unconnected-(U1-6_OUT1D-Pad8) -> Net-(U0-6_OUT1D)
- U1 pad 9: unconnected-(U1-7_RX2_OUT1A-Pad9) -> Net-(U0-7_RX2_OUT1A)
Routing:
- net AM0: track 29.0 -> 64.7 mm, vias 0 -> 2
- net AM0:2: track 11.9 -> 43.7 mm
- net GND: track 10.5 -> 36.8 mm, vias 0 -> 9
- net AM0:1: track 30.9 -> 45.9 mm
- net CONTROL3: track 22.8 -> 35.6 mm
- net CONTROL1: track 33.8 -> 43.9 mm
- net CONTROL2: track 26.6 -> 34.5 mm
- net +5V: track 47.2 -> 52.9 mm, vias 1 -> 0
- net CONTROL0: track 37.6 -> 42.9 mm
- net Net-(U1-41_A17): track 3.56 -> 0.00 mm
- net Net-(U0-41_A17): track 0.00 -> 3.32 mm
- net AM0:0: track 18.5 -> 21.4 mm
- net +3.3V: track 27.5 -> 29.6 mm, vias 7 -> 0
Other:
- board size 85 x 75 mm -> 77.5 x 63.5 mm

Commit message: Ok
Parts:
- AM0: footprint easyeda2kicad:SSOP-24_L8.1-W5.3-P0.65-LS7.8-BL -> jlcpcb:SSOP-24_L8.1-W5.3-P0.65-LS7.8-BL
- C0, C1, C2, C3: footprint easyeda2kicad:C0402 -> jlcpcb:C0402
- C4, C5: footprint easyeda2kicad:C0603 -> jlcpcb:C0603
- DC0: footprint easyeda2kicad:DC-IN-TH_DC-005-A250 -> jlcpcb:DC-IN-TH_DC-005-A250
- LDO1: footprint easyeda2kicad:TO-263-3_L8.6-W10.2-P2.54-LS14.4-TL -> jlcpcb:TO-263-3_L8.6-W10.2-P2.54-LS14.4-TL
- R0: footprint easyeda2kicad:R1206 -> jlcpcb:R1206
- S0, S1, S2: footprint easyeda2kicad:SOT-23-3_L2.9-W1.3-P1.90-LS2.4-BR -> jlcpcb:SOT-23-3_L2.9-W1.3-P1.90-LS2.4-BR
- U1, U2: footprint easyeda2kicad:HDR-TH_24P-P2.54-V-F -> jlcpcb:HDR-TH_24P-P2.54-V-F
Changed lines of the file:
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@@
 	(net 49 "Net-(U0-13_SCK_LED)")
 	(net 50 "Net-(U0-25_A11_RX6_SDA2)")
-	(footprint "easyeda2kicad:C0402"
+	(footprint "jlcpcb:C0402"
 		(layer "F.Cu")
 		(at 81.992 54.538371)
@@
 			)
 		)
-		(property "Footprint" "easyeda2kicad:C0402"
+		(property "Footprint" "jlcpcb:C0402"
 			(at 0 0 0)
 			(layer "F.Fab")
@@
 			(pintype "input")
 		)
-		(model "${EASYEDA2KICAD}/easyeda2kicad.3dshapes/C0402_L1.0-W0.5-H0.5.wrl"
+		(model "${EASYEDA2KICAD}/jlcpcb.3dshapes/C0402_L1.0-W0.5-H0.5.wrl"
 			(offset
 				(xyz 0 -0 -0)
@@
 		)
 	)
-	(footprint "easyeda2kicad:DC-IN-TH_DC-005-A250"
+	(footprint "jlcpcb:DC-IN-TH_DC-005-A250"
 		(layer "F.Cu")
 		(at 42.7625 63.1315)
@@
 			)
 		)
-		(property "Footprint" "easyeda2kicad:DC-IN-TH_DC-005-A250"
+		(property "Footprint" "jlcpcb:DC-IN-TH_DC-005-A250"
 			(at 0 0 0)
 			(layer "F.Fab")
@@
 			(pintype "unspecified")
 		)
-		(model "${EASYEDA2KICAD}/easyeda2kicad.3dshapes/DC-IN-TH_DC-005-A250.wrl"
+		(model "${EASYEDA2KICAD}/jlcpcb.3dshapes/DC-IN-TH_DC-005-A250.wrl"
 			(offset
 				(xyz -3.5 2.2 0)
@@
 		)
 	)
-	(footprint "easyeda2kicad:HDR-TH_24P-P2.54-V-F"
+	(footprint "jlcpcb:HDR-TH_24P-P2.54-V-F"
 		(layer "F.Cu")
 		(at 64.466 31.75)
@@
 			)
 		)
-		(property "Footprint" "easyeda2kicad:HDR-TH_24P-P2.54-V-F"
+		(property "Footprint" "jlcpcb:HDR-TH_24P-P2.54-V-F"
 			(at 0 0 0)
 			(layer "F.Fab")
@@
 			(pintype "unspecified")
 		)
-		(model "${EASYEDA2KICAD}/easyeda2kicad.3dshapes/HDR-TH_24P-P2.54-V-F.wrl"
+		(model "${EASYEDA2KICAD}/jlcpcb.3dshapes/HDR-TH_24P-P2.54-V-F.wrl"
 			(offset
 				(xyz 0 -0 0)
@@
 		)
 	)
-	(footprint "easyeda2kicad:HDR-TH_24P-P2.54-V-F"
+	(footprint "jlcpcb:HDR-TH_24P-P2.54-V-F"
 		(layer "F.Cu")
 		(at 64.466 46.99)
@@
 			)
 		)
-		(property "Footprint" "easyeda2kicad:HDR-TH_24P-P2.54-V-F"
+		(property "Footprint" "jlcpcb:HDR-TH_24P-P2.54-V-F"
 			(at 0 0 0)
 			(layer "F.Fab")
@@
 			(pintype "unspecified")
 		)
-		(model "${EASYEDA2KICAD}/easyeda2kicad.3dshapes/HDR-TH_24P-P2.54-V-F.wrl"
+		(model "${EASYEDA2KICAD}/jlcpcb.3dshapes/HDR-TH_24P-P2.54-V-F.wrl"
 			(offset
 				(xyz 0 -0 0)
@@
 		)
 	)
-	(footprint "easyeda2kicad:SSOP-24_L8.1-W5.3-P0.65-LS7.8-BL"
+	(footprint "jlcpcb:SSOP-24_L8.1-W5.3-P0.65-LS7.8-BL"
 		(layer "F.Cu")
 		(at 53.544 76.962)
@@
 			)
 		)
-		(property "Footprint" "easyeda2kicad:SSOP-24_L8.1-W5.3-P0.65-LS7.8-BL"
+		(property "Footprint" "jlcpcb:SSOP-24_L8.1-W5.3-P0.65-LS7.8-BL"
 			(at 0 0 0)
 			(layer "F.Fab")
@@
 			(pintype "unspecified")
 		)
-		(model "${EASYEDA2KICAD}/easyeda2kicad.3dshapes/SSOP-24_L8.2-W5.3-H1.8-LS7.8-P0.65.wrl"
+		(model "${EASYEDA2KICAD}/jlcpcb.3dshapes/SSOP-24_L8.2-W5.3-H1.8-LS7.8-P0.65.wrl"
 			(offset
 				(xyz 0 -0 -0)
@@
 		)
 	)
-	(footprint "easyeda2kicad:SOT-23-3_L2.9-W1.3-P1.90-LS2.4-BR"
+	(footprint "jlcpcb:SOT-23-3_L2.9-W1.3-P1.90-LS2.4-BR"
 		(layer "F.Cu")
 		(at 92.152 75.946)
@@
 			)
 		)
-		(property "Footprint" "easyeda2kicad:SOT-23-3_L2.9-W1.3-P1.90-LS2.4-BR"
+		(property "Footprint" "jlcpcb:SOT-23-3_L2.9-W1.3-P1.90-LS2.4-BR"
 			(at 0 0 0)
 			(layer "F.Fab")
@@
 			(pintype "unspecified")
 		)
-		(model "${EASYEDA2KICAD}/easyeda2kicad.3dshapes/SOT-23-3P_L2.9-W1.3-H1.0-LS2.4-P0.95.wrl"
+		(model "${EASYEDA2KICAD}/jlcpcb.3dshapes/SOT-23-3P_L2.9-W1.3-H1.0-LS2.4-P0.95.wrl"
 			(offset
 				(xyz -861.57 843.28 -0)
@@
 		)
 	)
-	(footprint "easyeda2kicad:SOT-23-3_L2.9-W1.3-P1.90-LS2.4-BR"
+	(footprint "jlcpcb:SOT-23-3_L2.9-W1.3-P1.90-LS2.4-BR"
 		(layer "F.Cu")
 		(at 71.832 75.946)
@@
 			)
 		)
-		(property "Footprint" "easyeda2kicad:SOT-23-3_L2.9-W1.3-P1.90-LS2.4-BR"
+		(property "Footprint" "jlcpcb:SOT-23-3_L2.9-W1.3-P1.90-LS2.4-BR"
 			(at 0 0 0)
 			(layer "F.Fab")
@@
 			(pintype "unspecified")
 		)
-		(model "${EASYEDA2KICAD}/easyeda2kicad.3dshapes/SOT-23-3P_L2.9-W1.3-H1.0-LS2.4-P0.95.wrl"
+		(model "${EASYEDA2KICAD}/jlcpcb.3dshapes/SOT-23-3P_L2.9-W1.3-H1.0-LS2.4-P0.95.wrl"
 			(offset
 				(xyz -861.57 843.28 -0)
@@
 		)
 	)
-	(footprint "easyeda2kicad:SOT-23-3_L2.9-W1.3-P1.90-LS2.4-BR"
+	(footprint "jlcpcb:SOT-23-3_L2.9-W1.3-P1.90-LS2.4-BR"
 		(layer "F.Cu")
 		(at 81.992 58.348371)
@@
 			)
 		)
-		(property "Footprint" "easyeda2kicad:SOT-23-3_L2.9-W1.3-P1.90-LS2.4-BR"
+		(property "Footprint" "jlcpcb:SOT-23-3_L2.9-W1.3-P1.90-LS2.4-BR"
 			(at 0 0 0)
 			(layer "F.Fab")
@@
 			(pintype "unspecified")
 		)
-		(model "${EASYEDA2KICAD}/easyeda2kicad.3dshapes/SOT-23-3P_L2.9-W1.3-H1.0-LS2.4-P0.95.wrl"
+		(model "${EASYEDA2KICAD}/jlcpcb.3dshapes/SOT-23-3P_L2.9-W1.3-H1.0-LS2.4-P0.95.wrl"
 			(offset
 				(xyz -861.57 843.28 -0)
@@
 		)
 	)
-	(footprint "easyeda2kicad:C0402"
+	(footprint "jlcpcb:C0402"
 		(layer "F.Cu")
 		(at 71.832 72.136)
@@
 			)
 		)
-		(property "Footprint" "easyeda2kicad:C0402"
+		(property "Footprint" "jlcpcb:C0402"
 			(at 0 0 0)
 			(layer "F.Fab")
@@
 			(pintype "input")
 		)
-		(model "${EASYEDA2KICAD}/easyeda2kicad.3dshapes/C0402_L1.0-W0.5-H0.5.wrl"
+		(model "${EASYEDA2KICAD}/jlcpcb.3dshapes/C0402_L1.0-W0.5-H0.5.wrl"
 			(offset
 				(xyz 0 -0 -0)
@@
 		)
 	)
-	(footprint "easyeda2kicad:TO-263-3_L8.6-W10.2-P2.54-LS14.4-TL"
+	(footprint "jlcpcb:TO-263-3_L8.6-W10.2-P2.54-LS14.4-TL"
 		(layer "F.Cu")
 		(at 62.18 58.42)
@@
 			)
 		)
-		(property "Footprint" "easyeda2kicad:TO-263-3_L8.6-W10.2-P2.54-LS14.4-TL"
+		(property "Footprint" "jlcpcb:TO-263-3_L8.6-W10.2-P2.54-LS14.4-TL"
 			(at 0 0 0)
 			(layer "F.Fab")
@@
 			(pintype "unspecified")
 		)
-		(model "${EASYEDA2KICAD}/easyeda2kicad.3dshapes/TO-263-3_4PIN-L8.6-W10.2-H4.8-P2.54-LS14.4-TL.wrl"
+		(model "${EASYEDA2KICAD}/jlcpcb.3dshapes/TO-263-3_4PIN-L8.6-W10.2-H4.8-P2.54-LS14.4-TL.wrl"
 			(offset
 				(xyz 1.98 -0 -0)
@@
 		)
 	)
-	(footprint "easyeda2kicad:R1206"
+	(footprint "jlcpcb:R1206"
 		(layer "F.Cu")
 		(at 74.88 28.448)
@@
 			)
 		)
-		(property "Footprint" "easyeda2kicad:R1206"
+		(property "Footprint" "jlcpcb:R1206"
 			(at 0 0 0)
 			(layer "F.Fab")
@@
 			(pintype "input")
 		)
-		(model "${EASYEDA2KICAD}/easyeda2kicad.3dshapes/R1206_L3.2-W1.6-H0.6.wrl"
+		(model "${EASYEDA2KICAD}/jlcpcb.3dshapes/R1206_L3.2-W1.6-H0.6.wrl"
 			(offset
 				(xyz -2.39 0.89 -0)
@@
 		)
 	)
-	(footprint "easyeda2kicad:C0402"
+	(footprint "jlcpcb:C0402"
 		(layer "F.Cu")
 		(at 49.988 71.12 90)
@@
 			)
 		)
-		(property "Footprint" "easyeda2kicad:C0402"
+		(property "Footprint" "jlcpcb:C0402"
 			(at 0 0 90)
 			(layer "F.Fab")
@@
 			(pintype "input")
 		)
-		(model "${EASYEDA2KICAD}/easyeda2kicad.3dshapes/C0402_L1.0-W0.5-H0.5.wrl"
+		(model "${EASYEDA2KICAD}/jlcpcb.3dshapes/C0402_L1.0-W0.5-H0.5.wrl"
 			(offset
 				(xyz 0 -0 -0)
@@
 		)
 	)
-	(footprint "easyeda2kicad:C0402"
+	(footprint "jlcpcb:C0402"
 		(layer "F.Cu")
 		(at 92.152 72.136)
@@
 			)
 		)
-		(property "Footprint" "easyeda2kicad:C0402"
+		(property "Footprint" "jlcpcb:C0402"
 			(at 0 0 0)
 			(layer "F.Fab")
@@
 			(pintype "input")
 		)
-		(model "${EASYEDA2KICAD}/easyeda2kicad.3dshapes/C0402_L1.0-W0.5-H0.5.wrl"
+		(model "${EASYEDA2KICAD}/jlcpcb.3dshapes/C0402_L1.0-W0.5-H0.5.wrl"
 			(offset
 				(xyz 0 -0 -0)
@@
 		)
 	)
-	(footprint "easyeda2kicad:C0603"
+	(footprint "jlcpcb:C0603"
 		(layer "F.Cu")
 		(at 52.274 63.308 -90)
@@
 			)
 		)
-		(property "Footprint" "easyeda2kicad:C0603"
+		(property "Footprint" "jlcpcb:C0603"
 			(at 0 0 90)
 			(layer "F.Fab")
@@
 			(pintype "unspecified")
 		)
-		(model "${EASYEDA2KICAD}/easyeda2kicad.3dshapes/C0603_L1.6-W0.8-H0.8.wrl"
+		(model "${EASYEDA2KICAD}/jlcpcb.3dshapes/C0603_L1.6-W0.8-H0.8.wrl"
 			(offset
 				(xyz -0.5 -0.13 -0)
@@
 		)
 	)
-	(footprint "easyeda2kicad:C0603"
+	(footprint "jlcpcb:C0603"
 		(layer "F.Cu")
 		(at 52.274 57.15 90)
@@
 			)
 		)
-		(property "Footprint" "easyeda2kicad:C0603"
+		(property "Footprint" "jlcpcb:C0603"
 			(at 0 0 90)
 			(layer "F.Fab")
@@
 			(pintype "unspecified")
 		)
-		(model "${EASYEDA2KICAD}/easyeda2kicad.3dshapes/C0603_L1.6-W0.8-H0.8.wrl"
+		(model "${EASYEDA2KICAD}/jlcpcb.3dshapes/C0603_L1.6-W0.8-H0.8.wrl"
 			(offset
 				(xyz -0.5 -0.13 -0)

Commit message: Ok
Routing:
- net GND: track 36.8 -> 42.9 mm
Changed lines of the file:
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@@
 		(legacy_teardrops no)
 	)
-	(paper "A4")
+	(paper "A5")
 	(layers
 		(0 "F.Cu" signal)
@@
 			(sketchpadsonfab no)
 			(subtractmaskfromsilk no)
-			(outputformat 1)
+			(outputformat 4)
 			(mirror no)
-			(drillshape 1)
+			(drillshape 0)
 			(scaleselection 1)
-			(outputdirectory "")
+			(outputdirectory "../../../../Documents/")
 		)
 	)
@@
 			(at 0 -4 0)
 			(layer "F.SilkS")
+			(hide yes)
 			(effects
 				(font
@@
 			(at 0 4 0)
 			(layer "F.Fab")
+			(hide yes)
 			(effects
 				(font
@@
 		)
 		(fp_text user "${REFERENCE}"
-			(at 0 0 0)
+			(at 0 -1.325371 0)
 			(layer "F.Fab")
 			(effects
@@
 			(at 0 -6.33 0)
 			(layer "F.SilkS")
+			(hide yes)
 			(effects
 				(font
@@
 			(at 0 6.32 0)
 			(layer "F.Fab")
+			(hide yes)
 			(effects
 				(font
@@
 			(at 0 4.2 0)
 			(layer "F.Fab")
+			(hide yes)
 			(effects
 				(font
@@
 			(at 0 4.2 0)
 			(layer "F.Fab")
+			(hide yes)
 			(effects
 				(font
@@
 			(at 0 4.2 0)
 			(layer "F.Fab")
+			(hide yes)
 			(effects
 				(font
@@
 			(at 0 -7.56 0)
 			(layer "F.SilkS")
+			(hide yes)
 			(effects
 				(font
@@
 			(at 0 7.56 0)
 			(layer "F.Fab")
+			(hide yes)
 			(effects
 				(font
@@
 			(at 0 -4.95 0)
 			(layer "F.SilkS")
+			(hide yes)
 			(effects
 				(font
@@
 			(at 0 4.95 0)
 			(layer "F.Fab")
+			(hide yes)
 			(effects
 				(font
@@
 		)
 		(fp_text user "${REFERENCE}"
-			(at 0 0 0)
+			(at 0.05 3.302 0)
 			(layer "F.Fab")
 			(effects
@@
 			(at 0 -4.95 0)
 			(layer "F.SilkS")
+			(hide yes)
 			(effects
 				(font
@@
 			(at 0 4.95 0)
 			(layer "F.Fab")
+			(hide yes)
 			(effects
 				(font
@@
 		)
 		(fp_text user "${REFERENCE}"
-			(at 0 0 0)
+			(at -0.204 3.302 0)
 			(layer "F.Fab")
 			(effects
@@
 			(at 0 -4.95 0)
 			(layer "F.SilkS")
+			(hide yes)
 			(effects
 				(font
@@
 			(at 0 4.95 0)
 			(layer "F.Fab")
+			(hide yes)
 			(effects
 				(font
@@
 		)
 		(fp_text user "${REFERENCE}"
-			(at 0 0 0)
+			(at -0.077 3.373629 0)
 			(layer "F.Fab")
 			(effects
@@
 			(at 0 -4 0)
 			(layer "F.SilkS")
+			(hide yes)
 			(effects
 				(font
@@
 			(at 0 4 0)
 			(layer "F.Fab")
+			(hide yes)
 			(effects
 				(font
@@
 		)
 		(fp_text user "${REFERENCE}"
-			(at 0 0 0)
+			(at 0 -1.397 0)
 			(layer "F.Fab")
 			(effects
@@
 			(at 0 -6.54 0)
 			(layer "F.SilkS")
+			(hide yes)
 			(effects
 				(font
@@
 			(at 0 6.54 0)
 			(layer "F.Fab")
+			(hide yes)
 			(effects
 				(font
@@
 		)
 		(fp_text user "${REFERENCE}"
-			(at 0 0 0)
+			(at 0.05 -6.985 0)
 			(layer "F.Fab")
 			(effects
@@
 			(at 0 -4 0)
 			(layer "F.SilkS")
+			(hide yes)
 			(effects
 				(font
@@
 			(at 0 4 0)
 			(layer "F.Fab")
+			(hide yes)
 			(effects
 				(font
@@
 			(at 0 -4 90)
 			(layer "F.SilkS")
+			(hide yes)
 			(effects
 				(font
@@
 			(at 0 4 90)
 			(layer "F.Fab")
+			(hide yes)
 			(effects
 				(font
@@
 		)
 		(fp_text user "${REFERENCE}"
-			(at 0 0 90)
+			(at 0 -1.474 90)
 			(layer "F.Fab")
 			(effects
@@
 			(at 0 -4 0)
 			(layer "F.SilkS")
+			(hide yes)
 			(effects
 				(font
@@
 			(at 0 4 0)
 			(layer "F.Fab")
+			(hide yes)
 			(effects
 				(font
@@
 		)
 		(fp_text user "${REFERENCE}"
-			(at 0 0 0)
+			(at 0.05 -1.143 0)
 			(layer "F.Fab")
 			(effects
@@
 			(at 0 4.2 0)
 			(layer "F.Fab")
+			(hide yes)
 			(effects
 				(font
@@
 			(at 0 -4 90)
 			(layer "F.SilkS")
+			(hide yes)
 			(effects
 				(font
@@
 			(at 0 4 90)
 			(layer "F.Fab")
+			(hide yes)
 			(effects
 				(font
@@
 		)
 		(fp_text user "${REFERENCE}"
-			(at -0.062 1.347 90)
+			(at 0.065 1.728 90)
 			(layer "F.Fab")
 			(effects
@@
 			(at 0 -4 90)
 			(layer "F.SilkS")
+			(hide yes)
 			(effects
 				(font
@@
 			(at 0 4 90)
 			(layer "F.Fab")
+			(hide yes)
 			(effects
 				(font
@@
 		)
 		(fp_text user "${REFERENCE}"
-			(at 0.127 -1.22 90)
+			(at 0 -1.601 90)
 			(layer "F.Fab")
 			(effects
@@
 			(at 0 3.048 0)
 			(layer "Dwgs.User")
+			(hide yes)
 			(effects
 				(font
@@
 		(fp_arc
 			(start 6.497236 -6.998884)
-			(mid 6.85079 -6.852453)
+			(mid 6.850825 -6.852459)
 			(end 6.997236 -6.498884)
 			(stroke
@@
 			(at 0 3.048 0)
 			(layer "Dwgs.User")
+			(hide yes)
 			(effects
 				(font
@@
 		(fp_arc
 			(start 6.497236 -6.998884)
-			(mid 6.85079 -6.852453)
+			(mid 6.850825 -6.852459)
 			(end 6.997236 -6.498884)
 			(stroke
@@
 			(at 0 3.048 0)
 			(layer "Dwgs.User")
+			(hide yes)
 			(effects
 				(font
@@
 		(fp_arc
 			(start 6.497236 -6.998884)
-			(mid 6.85079 -6.852453)
+			(mid 6.850825 -6.852459)
 			(end 6.997236 -6.498884)
 			(stroke
@@
 		(net 4)
 	)
+	(segment
+		(start 39.7625 60.8015)
+		(end 39.7625 61.9515)
+		(width 1.524)
+		(layer "B.Cu")
+		(net 4)
+	)
+	(segment
+		(start 39.7625 61.9515)
+		(end 43.2625 65.4515)
+		(width 1.524)
+		(layer "B.Cu")
+		(net 4)
+	)

Commit message: Ok
Parts:
- removed AM0: CD74HC4067SM96, jlcpcb:SSOP-24_L8.1-W5.3-P0.65-LS7.8-BL
- removed C0: CL05B104KA5NNNC, jlcpcb:C0402
- removed DC0: DC-005-A250, jlcpcb:DC-IN-TH_DC-005-A250
- removed LDO1: AMS1085CM-3.3, jlcpcb:TO-263-3_L8.6-W10.2-P2.54-LS14.4-TL
- removed R0: 1206W4F1001T5E, jlcpcb:R1206
- removed REF0: SW_MX_Lekker, lekker:SW_MX_Lekker
- removed S0: GH39FKSW, jlcpcb:SOT-23-3_L2.9-W1.3-P1.90-LS2.4-BR
- removed U1, U2: X6511FV-24-C85D32, jlcpcb:HDR-TH_24P-P2.54-V-F
- added AM1: CD74HC4067SM96, jlcpcb:SSOP-24_L8.1-W5.3-P0.65-LS7.8-BL, F.Cu at (82.2, 69.2)
- added C6: 100 nF, jlcpcb:C0603, F.Cu at (78.6, 49.5)
- added C7: 220 pF, jlcpcb:C0603, F.Cu at (76.4, 57.9)
- added C8: 22 uF, jlcpcb:C1206, F.Cu at (74.8, 50.2)
- added C9: 22 uF, jlcpcb:C1206, F.Cu at (72.3, 50.2)
- added DC1: DC-005-A250, jlcpcb:DC-IN-TH_DC-005-A250, B.Cu at (88.2, 55.0)
- added J1: X6511FV-24-C85D32, jlcpcb:HDR-TH_24P-P2.54-V-F, B.Cu at (68.7, 39.0)
- added J2: X6511FV-24-C85D32, jlcpcb:HDR-TH_24P-P2.54-V-F, B.Cu at (68.7, 23.7)
- added L1: 4.7 uH, jlcpcb:IND-SMD_L4.1-W4.1_SPM40XX, F.Cu at (78.5, 46.4)
- added R1: 100 kΩ, jlcpcb:R0603, F.Cu at (76.5, 56.2)
- added R2: 22.1 kΩ, jlcpcb:R0603, F.Cu at (76.4, 54.5)
- added R3: 1k, jlcpcb:R1206, F.Cu at (62.0, 27.9)
- added REF3: KEY3, lekker:SW_MX_Lekker, B.Cu at (46.7, 66.9)
- added S3: GH39FKSW, jlcpcb:SOT-23-3_L2.9-W1.3-P1.90-LS2.4-BR, F.Cu at (46.7, 66.9)
- added VR1: SY8113IADC, jlcpcb:TSOT-23-6_L2.9-W1.6-P0.95-LS2.8-BL, F.Cu at (78.4, 52.1)
- C1, C2, C3: value CL05B104KA5NNNC -> 100 nF; footprint jlcpcb:C0402 -> jlcpcb:C0603
- C4: value CL10A106MQ8NNNC -> 100 nF
- C5: value CL10A106MQ8NNNC -> 10 uF; footprint jlcpcb:C0603 -> jlcpcb:C0805
- FID1, FID2, FID3: value Fiducial -> Fiducial_1mm_Mask2mm
- REF1: value SW_MX_Lekker -> KEY1
- REF2: value SW_MX_Lekker -> KEY2
- moved H3 65.2 mm to (95.2, 71.6)
- moved C2 44.2 mm to (56.9, 45.5)
- moved REF2 44.2 mm to (56.9, 49.3)
- moved S2 44.2 mm to (56.9, 49.3)
- moved FID3 38.9 mm to (100.6, 66.9)
- moved C4 34.4 mm to (84.8, 74.4), turned to 0 degrees
- moved C5 29.8 mm to (81.8, 53.3)
- moved H4 26.6 mm to (56.9, 59.7)
- moved FID2 23.4 mm to (86.4, 29.2)
- moved FID1 20.4 mm to (41.9, 50.8)
- moved C1 17.2 mm to (67.1, 63.1)
- moved REF1 17.2 mm to (67.1, 66.9)
- moved S1 17.2 mm to (67.1, 66.9)
- moved H1 13.3 mm to (42.4, 31.5)
- moved C3 8.64 mm to (46.7, 63.1), turned to 0 degrees
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Connections:
- C1 pad 1: +3.3V -> GND
- C1 pad 2: GND -> +3.3V
- C2 pad 1: +3.3V -> GND
- C2 pad 2: GND -> +3.3V
- C3 pad 1: +3.3V -> GND
- C3 pad 2: GND -> +3.3V
- C4 pad 1: +5V -> GND
- C4 pad 2: GND -> +3.3V
- C5 pad 1: +3.3V -> GND
- C5 pad 2: GND -> +5V
- S1 pad 2: AM0:1 -> AM1:0
- S2 pad 2: AM0:2 -> AM1:1
Routing:
- net AM0: track 64.7 -> 0.00 mm, vias 2 -> 0
- net AM1: track 0.00 -> 58.3 mm, vias 0 -> 2
- net AM0:1: track 45.9 -> 0.00 mm
- net AM0:2: track 43.7 -> 0.00 mm
- net AM1:2: track 0.00 -> 40.1 mm
- net AM1:1: track 0.00 -> 30.9 mm
- net +3.3V: track 29.6 -> 7.55 mm
- net AM0:0: track 21.4 -> 0.00 mm
- net AM1:0: track 0.00 -> 15.8 mm
- net +5V: track 52.9 -> 46.0 mm
- net CONTROL2: track 34.5 -> 39.7 mm
- net Net-(VR1-LX): track 0.00 -> 5.20 mm
- net CONTROL3: track 35.6 -> 40.8 mm
- net Net-(VR1-FB): track 0.00 -> 4.92 mm
- net Net-(J2-41_A17): track 0.00 -> 4.49 mm
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- added copper zone on F.Cu, net +5V
- added copper zone on F.Cu, net GND
Other:
- board size 77.5 x 63.5 mm -> 73.7 x 61 mm
- board text added: "github.com/DumpsterDoofus/keyboard_accordion (3_key V1)"
