File: kicad/3_key/3_key.kicad_pcb (KiCad board)
At the start: 2 copper layers, 73.7 x 61 mm, 31 parts, among them J1 X6511FV-24-C85D32, J2 X6511FV-24-C85D32

Commit message: 3_key v1
Parts:
- removed C6: 100 nF, jlcpcb:C0603
- removed C7: 220 pF, jlcpcb:C0603
- removed C8, C9: 22 uF, jlcpcb:C1206
- removed L1: 4.7 uH, jlcpcb:IND-SMD_L4.1-W4.1_SPM40XX
- removed REF1: KEY1, lekker:SW_MX_Lekker
- removed REF2: KEY2, lekker:SW_MX_Lekker
- removed REF3: KEY3, lekker:SW_MX_Lekker
- removed VR1: SY8113IADC, jlcpcb:TSOT-23-6_L2.9-W1.6-P0.95-LS2.8-BL
- added H5: MountingHole, MountingHole:MountingHole_3.2mm_M3_Pad, F.Cu at (57.7, 60.1)
- added KEY1: SW_MX_Lekker, lekker:SW_MX_Lekker, B.Cu at (47.5, 67.5)
- added KEY2: SW_MX_Lekker, lekker:SW_MX_Lekker, B.Cu at (67.8, 67.5)
- added KEY3: SW_MX_Lekker, lekker:SW_MX_Lekker, B.Cu at (57.7, 49.9)
- C5: value 10 uF -> 22 uF; footprint jlcpcb:C0805 -> jlcpcb:C1206
- DC1, J1, J2: moved to F.Cu
- R1: value 100 kΩ -> 1k; footprint jlcpcb:R0603 -> jlcpcb:R1206
- R2: value 22.1 kΩ -> 1k; footprint jlcpcb:R0603 -> jlcpcb:R1206
- moved H3 71.8 mm to (23.5, 73.0)
- moved C4 50.3 mm to (39.8, 52.0)
- moved AM1 49.2 mm to (38.9, 46.0)
- moved R1 45.6 mm to (35.5, 36.1), turned to 0 degrees
- moved H4 35.3 mm to (89.5, 73.0)
- moved C2 28.0 mm to (67.8, 71.3)
- moved H1 22.3 mm to (23.5, 19.7)
- moved R3 21.8 mm to (74.5, 45.8), turned to -90 degrees
- moved S2 21.2 mm to (67.8, 67.5)
- moved C1 21.2 mm to (47.5, 71.3)
- moved S3 20.3 mm to (57.7, 49.9)
- moved J2 19.8 mm to (56.2, 39.1)
- moved J1 19.7 mm to (56.2, 23.8)
- moved S1 19.5 mm to (47.5, 67.5)
- moved R2 19.1 mm to (81.5, 36.1)
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Connections:
- AM1 pad 15: GND -> ENABLE
- AM1 pad 7: AM1:0 -> AM1:2
- AM1 pad 8: AM1:2 -> AM1:1
- AM1 pad 9: AM1:1 -> AM1:0
- C5 pad 2: +5V -> +3.3V
- DC1 pad 1: +5V -> +3.3V
- J1 pad 4: CONTROL0 -> unconnected-(J1-2_OUT2-Pad4)
- J1 pad 5: CONTROL1 -> unconnected-(J1-3_LRCLK2-Pad5)
- J1 pad 6: CONTROL2 -> unconnected-(J1-4_BCLK2-Pad6)
- J1 pad 7: CONTROL3 -> unconnected-(J1-5_IN2-Pad7)
- J2 pad 16: Net-(J2-41_A17) -> unconnected-(J2-41_A17-Pad16)
- J2 pad 20: unconnected-(J2-37_CS-Pad20) -> Net-(J2-37_CS)
- J2 pad 21: unconnected-(J2-36_CS-Pad21) -> CONTROL2
- J2 pad 22: unconnected-(J2-35_TX8-Pad22) -> CONTROL3
- J2 pad 23: unconnected-(J2-34_RX8-Pad23) -> CONTROL0
- J2 pad 24: unconnected-(J2-33_MCLK2-Pad24) -> CONTROL1
- J2 pad 3: unconnected-(J2-3V3-Pad3) -> ENABLE
- R1 pad 1: Net-(VR1-FB) -> +3.3V
- R1 pad 2: +3.3V -> Net-(J2-37_CS)
- R2 pad 1: GND -> ENABLE
- R2 pad 2: Net-(VR1-FB) -> GND
- R3 pad 1: Net-(J2-41_A17) -> GND
Routing:
- net ENABLE: track 0.00 -> 52.2 mm, vias 0 -> 1
- net +5V: track 46.0 -> 0.00 mm
- net AM1: track 58.3 -> 18.9 mm, vias 2 -> 0
- net CONTROL2: track 39.7 -> 4.17 mm
- net CONTROL3: track 40.8 -> 6.02 mm
- net CONTROL1: track 45.2 -> 13.9 mm
- net CONTROL0: track 44.1 -> 13.1 mm
- net AM1:2: track 40.1 -> 23.6 mm
- net AM1:0: track 15.8 -> 29.5 mm
- net GND: track 40.9 -> 54.4 mm, vias 11 -> 5
- net AM1:1: track 30.9 -> 43.7 mm
- net +3.3V: track 7.55 -> 15.5 mm
- net Net-(VR1-LX): track 5.20 -> 0.00 mm
- net Net-(VR1-FB): track 4.92 -> 0.00 mm
- net Net-(J2-41_A17): track 4.49 -> 0.00 mm
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- removed copper zone on F.Cu, net +5V
- removed copper zone on F.Cu, net GND
Other:
- board size 73.7 x 61 mm -> 74.9 x 62.2 mm
