File: hardware/kicad/96_key/96_key.kicad_sch (KiCad schematic)
At the start: 205 parts, among them U1 PM254-1-14-W-8.5

Commit message: Replace C98457 (out of stock) with C179326
Parts:
- AM0, AM1, AM2, AM3, AM4, AM5: footprint jlcpcb:SSOP-24_L8.1-W5.3-P0.65-LS7.8-BL -> jlcpcb:TSSOP-24_L7.8-W4.4-P0.65-LS6.4-BL; symbol jlcpcb:CD74HC4067SM96 -> jlcpcb:74HC4067PW,118; LCSC Part C98457 -> C179326
Other:
- moved on the sheet: C192, C193, C194, C195, C196, C197
