File: hardware/kicad/96_key/96_key.kicad_sch (KiCad schematic)
At the start: 205 parts, among them U1 PM254-1-14-W-8.5

Commit message: Feedback https://www.reddit.com/r/KiCad/comments/1pkh416/review_request_192key_hall_effect_keyboard
Changed lines of the file:
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@@
 	)
 	(junction
+		(at 71.12 76.2)
+		(diameter 0)
+		(color 0 0 0 0)
+	)
+	(junction
 		(at 521.97 49.53)
 		(diameter 0)
@@
 	(wire
 		(pts
+			(xy 71.12 76.2) (xy 74.93 76.2)
+		)
+		(stroke
+			(width 0)
+			(type default)
+		)
+	)
+	(wire
+		(pts
 			(xy 478.79 119.38) (xy 488.95 119.38)
 		)
@@
 	(wire
 		(pts
-			(xy 60.96 76.2) (xy 74.93 76.2)
+			(xy 60.96 76.2) (xy 71.12 76.2)
 		)
 		(stroke
@@
 					(unit 1)
 				)
+			)
+		)
+	)
+	(symbol
+		(lib_id "power:PWR_FLAG")
+		(at 71.12 76.2 0)
+		(unit 1)
+		(exclude_from_sim no)
+		(in_bom yes)
+		(on_board yes)
+		(dnp no)
+		(fields_autoplaced yes)
+		(property "Reference" "#FLG01"
+			(at 71.12 74.295 0)
+			(effects
+				(font
+					(size 1.27 1.27)
+				)
+				(hide yes)
+			)
+		)
+		(property "Value" "PWR_FLAG"
+			(at 71.12 71.12 0)
+			(effects
+				(font
+					(size 1.27 1.27)
+				)
+			)
+		)
+		(property "Footprint" ""
+			(at 71.12 76.2 0)
+			(effects
+				(font
+					(size 1.27 1.27)
+				)
+				(hide yes)
+			)
+		)
+		(property "Datasheet" "~"
+			(at 71.12 76.2 0)
+			(effects
+				(font
+					(size 1.27 1.27)
+				)
+				(hide yes)
+			)
+		)
+		(property "Description" "Special symbol for telling ERC where power comes from"
+			(at 71.12 76.2 0)
+			(effects
+				(font
+					(size 1.27 1.27)
+				)
+				(hide yes)
+			)
+		)
+		(pin "1"
+		)
+		(instances
+			(project "96_key"
+				(path "/3c4fbca4-0f94-4fe8-ac2f-7c937d86bae4"
+					(reference "#FLG01")
+					(unit 1)
+				)

Commit message: Ok
Parts:
- AM0, AM1, AM2, AM3, AM4, AM5: footprint jlcpcb:SSOP-24_L8.1-W5.3-P0.65-LS7.8-BL -> jlcpcb:TSSOP-24_L7.8-W4.4-P0.65-LS6.4-BL; symbol jlcpcb:CD74HC4067SM96 -> jlcpcb:74HC4067PW,118; LCSC Part C98457 -> C179326
Other:
- moved on the sheet: C192, C193, C194, C195, C196, C197

Commit message: Ok
Parts:
- AM0, AM1, AM2, AM3, AM4, AM5: value CD74HC4067SM96 -> 74HC4067PW,118
Other:
- title: (none) -> https://github.com/DumpsterDoofus/keyboard_accordion
- moved on the sheet: AM0, AM1, AM2, AM3, AM4, AM5, C0, C1, C10, C11, C12, C13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

Commit message: Ok
Parts:
- renumbered AM0 to AM1, AM1 to AM2, AM2 to AM3, AM3 to AM4, AM4 to AM5, AM5 to AM6, C0 to C1, C9 to C10, C195 to C100, C196 to C101, C197 to C102, C10 to C11, C11 to C12, C12 to C13, C13 to C14, C14 to C15, C15 to C16, C16 to C17, C17 to C18, C18 to C19, C1 to C2, C19 to C20, C20 to C21, C21 to C22, C22 to C23, C23 to C24, C24 to C25, C25 to C26, C26 to C27, C27 to C28, C28 to C29, C2 to C3, C29 to C30, C30 to C31, C31 to C32, C32 to C33, C33 to C34, C34 to C35, C35 to C36, C36 to C37, C37 to C38, C38 to C39, C3 to C4, C39 to C40, C40 to C41, C41 to C42, C42 to C43, C43 to C44, C44 to C45, C45 to C46, C46 to C47, C47 to C48, C48 to C49, C4 to C5, C49 to C50, C50 to C51, C51 to C52, C52 to C53, C53 to C54, C54 to C55, C55 to C56, C56 to C57, C57 to C58, C58 to C59, C5 to C6, C59 to C60, C60 to C61, C61 to C62, C62 to C63, C63 to C64, C64 to C65, C65 to C66, C66 to C67, C67 to C68, C68 to C69, C6 to C7, C69 to C70, C70 to C71, C71 to C72, C72 to C73, C73 to C74, C74 to C75, C75 to C76, C76 to C77, C77 to C78, C78 to C79, C7 to C8, C79 to C80, C80 to C81, C81 to C82, C82 to C83, C83 to C84, C84 to C85, C85 to C86, C86 to C87, C87 to C88, C88 to C89, C8 to C9, C89 to C90, C90 to C91, C91 to C92, C92 to C93, C93 to C94, C94 to C95, C95 to C96, C192 to C97, C193 to C98, C194 to C99, S0 to S1, S9 to S10, S10 to S11, S11 to S12, S12 to S13, S13 to S14, S14 to S15, S15 to S16, S16 to S17, S17 to S18, S18 to S19, S1 to S2, S19 to S20, S20 to S21, S21 to S22, S22 to S23, S23 to S24, S24 to S25, S25 to S26, S26 to S27, S27 to S28, S28 to S29, S2 to S3, S29 to S30, S30 to S31, S31 to S32, S32 to S33, S33 to S34, S34 to S35, S35 to S36, S36 to S37, S37 to S38, S38 to S39, S3 to S4, S39 to S40, S40 to S41, S41 to S42, S42 to S43, S43 to S44, S44 to S45, S45 to S46, S46 to S47, S47 to S48, S48 to S49, S4 to S5, S49 to S50, S50 to S51, S51 to S52, S52 to S53, S53 to S54, S54 to S55, S55 to S56, S56 to S57, S57 to S58, S58 to S59, S5 to S6, S59 to S60, S60 to S61, S61 to S62, S62 to S63, S63 to S64, S64 to S65, S65 to S66, S66 to S67, S67 to S68, S68 to S69, S6 to S7, S69 to S70, S70 to S71, S71 to S72, S72 to S73, S73 to S74, S74 to S75, S75 to S76, S76 to S77, S77 to S78, S78 to S79, S7 to S8, S79 to S80, S80 to S81, S81 to S82, S82 to S83, S83 to S84, S84 to S85, S85 to S86, S86 to S87, S87 to S88, S88 to S89, S8 to S9, S89 to S90, S90 to S91, S91 to S92, S92 to S93, S93 to S94, S94 to S95, S95 to S96
Connections:
- net AM0 is gone; now on net AM1: AM1.1 (Z), U1.10
- net AM0:0 is gone; now on net AM1:1: AM1.9 (Y0), S1.2 (VOUT)
- net AM0:1 is gone; now on net AM1:2: AM1.8 (Y1), S2.2 (VOUT)
- net AM0:10 is gone; now on net AM1:11: AM1.21 (Y10), S11.2 (VOUT)
- net AM0:11 is gone; now on net AM1:12: AM1.20 (Y11), S12.2 (VOUT)
- net AM0:12 is gone; now on net AM1:13: AM1.19 (Y12), S13.2 (VOUT)
- net AM0:13 is gone; now on net AM1:14: AM1.18 (Y13), S14.2 (VOUT)
- net AM0:14 is gone; now on net AM1:15: AM1.17 (Y14), S15.2 (VOUT)
- net AM0:2 is gone; now on net AM1:3: AM1.7 (Y2), S3.2 (VOUT)
- net AM0:3 is gone; now on net AM1:4: AM1.6 (Y3), S4.2 (VOUT)
- net AM0:4 is gone; now on net AM1:5: AM1.5 (Y4), S5.2 (VOUT)
- net AM0:5 is gone; now on net AM1:6: AM1.4 (Y5), S6.2 (VOUT)
- net AM0:6 is gone; now on net AM1:7: AM1.3 (Y6), S7.2 (VOUT)
- net AM0:7 is gone; now on net AM1:8: AM1.2 (Y7), S8.2 (VOUT)
- net AM0:8 is gone; now on net AM1:9: AM1.23 (Y8), S9.2 (VOUT)
- net AM0:9 is gone; now on net AM1:10: AM1.22 (Y9), S10.2 (VOUT)
- net AM1:0 is gone; now on net AM2:1: AM2.9 (Y0), S17.2 (VOUT)
- net AM2:0 is gone; now on net AM3:1: AM3.9 (Y0), S33.2 (VOUT)
- net AM3:0 is gone; now on net AM4:1: AM4.9 (Y0), S49.2 (VOUT)
- net AM4:0 is gone; now on net AM5:1: AM5.9 (Y0), S65.2 (VOUT)
- net CONTROL0 is gone; now on net CONTROL1: AM1.10 (S1), AM2.10 (S1), AM3.10 (S1), AM4.10 (S1), AM5.10 (S1), AM6.10 (S1), U1.11
- net AM1: no longer AM2.1 (Z), U1.9
- net AM1:1: no longer AM2.8 (Y1), S18.2 (VOUT)
- net AM1:10: no longer AM2.21 (Y10), S27.2 (VOUT)
- net AM1:11: no longer AM2.20 (Y11), S28.2 (VOUT)
- net AM1:12: no longer AM2.19 (Y12), S29.2 (VOUT)
- net AM1:13: no longer AM2.18 (Y13), S30.2 (VOUT)
- net AM1:14: no longer AM2.17 (Y14), S31.2 (VOUT)
- net AM1:15: no longer AM2.16 (Y15), S32.2 (VOUT)
- net AM1:2: no longer AM2.7 (Y2), S19.2 (VOUT)
- net AM1:3: no longer AM2.6 (Y3), S20.2 (VOUT)
- net AM1:4: no longer AM2.5 (Y4), S21.2 (VOUT)
- net AM1:5: no longer AM2.4 (Y5), S22.2 (VOUT)
- net AM1:6: no longer AM2.3 (Y6), S23.2 (VOUT)
- net AM1:7: no longer AM2.2 (Y7), S24.2 (VOUT)
- net AM1:8: no longer AM2.23 (Y8), S25.2 (VOUT)
- net AM1:9: no longer AM2.22 (Y9), S26.2 (VOUT)
- net AM2: now also AM2.1 (Z), U1.9; no longer AM3.1 (Z), U1.8
- net AM2:1: no longer AM3.8 (Y1), S34.2 (VOUT)
- net AM2:10: now also AM2.22 (Y9), S26.2 (VOUT); no longer AM3.21 (Y10), S43.2 (VOUT)
- net AM2:11: now also AM2.21 (Y10), S27.2 (VOUT); no longer AM3.20 (Y11), S44.2 (VOUT)
- net AM2:12: now also AM2.20 (Y11), S28.2 (VOUT); no longer AM3.19 (Y12), S45.2 (VOUT)
- net AM2:13: now also AM2.19 (Y12), S29.2 (VOUT); no longer AM3.18 (Y13), S46.2 (VOUT)
- net AM2:14: now also AM2.18 (Y13), S30.2 (VOUT); no longer AM3.17 (Y14), S47.2 (VOUT)
- net AM2:15: now also AM2.17 (Y14), S31.2 (VOUT); no longer AM3.16 (Y15), S48.2 (VOUT)
- net AM2:2: now also AM2.8 (Y1), S18.2 (VOUT); no longer AM3.7 (Y2), S35.2 (VOUT)
- net AM2:3: now also AM2.7 (Y2), S19.2 (VOUT); no longer AM3.6 (Y3), S36.2 (VOUT)
- net AM2:4: now also AM2.6 (Y3), S20.2 (VOUT); no longer AM3.5 (Y4), S37.2 (VOUT)
- net AM2:5: now also AM2.5 (Y4), S21.2 (VOUT); no longer AM3.4 (Y5), S38.2 (VOUT)
- net AM2:6: now also AM2.4 (Y5), S22.2 (VOUT); no longer AM3.3 (Y6), S39.2 (VOUT)
- net AM2:7: now also AM2.3 (Y6), S23.2 (VOUT); no longer AM3.2 (Y7), S40.2 (VOUT)
- net AM2:8: now also AM2.2 (Y7), S24.2 (VOUT); no longer AM3.23 (Y8), S41.2 (VOUT)
- net AM2:9: now also AM2.23 (Y8), S25.2 (VOUT); no longer AM3.22 (Y9), S42.2 (VOUT)
- net AM3: now also AM3.1 (Z), U1.8; no longer AM4.1 (Z), U1.5
- net AM3:1: no longer AM4.8 (Y1), S50.2 (VOUT)
- net AM3:10: now also AM3.22 (Y9), S42.2 (VOUT); no longer AM4.21 (Y10), S59.2 (VOUT)
- net AM3:11: now also AM3.21 (Y10), S43.2 (VOUT); no longer AM4.20 (Y11), S60.2 (VOUT)
- net AM3:12: now also AM3.20 (Y11), S44.2 (VOUT); no longer AM4.19 (Y12), S61.2 (VOUT)
- net AM3:13: now also AM3.19 (Y12), S45.2 (VOUT); no longer AM4.18 (Y13), S62.2 (VOUT)
- net AM3:14: now also AM3.18 (Y13), S46.2 (VOUT); no longer AM4.17 (Y14), S63.2 (VOUT)
- net AM3:15: now also AM3.17 (Y14), S47.2 (VOUT); no longer AM4.16 (Y15), S64.2 (VOUT)
- net AM3:2: now also AM3.8 (Y1), S34.2 (VOUT); no longer AM4.7 (Y2), S51.2 (VOUT)
- net AM3:3: now also AM3.7 (Y2), S35.2 (VOUT); no longer AM4.6 (Y3), S52.2 (VOUT)
- net AM3:4: now also AM3.6 (Y3), S36.2 (VOUT); no longer AM4.5 (Y4), S53.2 (VOUT)
- net AM3:5: now also AM3.5 (Y4), S37.2 (VOUT); no longer AM4.4 (Y5), S54.2 (VOUT)
- net AM3:6: now also AM3.4 (Y5), S38.2 (VOUT); no longer AM4.3 (Y6), S55.2 (VOUT)
- net AM3:7: now also AM3.3 (Y6), S39.2 (VOUT); no longer AM4.2 (Y7), S56.2 (VOUT)
- net AM3:8: now also AM3.2 (Y7), S40.2 (VOUT); no longer AM4.23 (Y8), S57.2 (VOUT)
- net AM3:9: now also AM3.23 (Y8), S41.2 (VOUT); no longer AM4.22 (Y9), S58.2 (VOUT)
- net AM4: now also AM4.1 (Z), U1.5; no longer AM5.1 (Z), U1.6
- net AM4:1: no longer AM5.8 (Y1), S66.2 (VOUT)
- net AM4:10: now also AM4.22 (Y9), S58.2 (VOUT); no longer AM5.21 (Y10), S75.2 (VOUT)
- net AM4:11: now also AM4.21 (Y10), S59.2 (VOUT); no longer AM5.20 (Y11), S76.2 (VOUT)
- net AM4:12: now also AM4.20 (Y11), S60.2 (VOUT); no longer AM5.19 (Y12), S77.2 (VOUT)
- net AM4:13: now also AM4.19 (Y12), S61.2 (VOUT); no longer AM5.18 (Y13), S78.2 (VOUT)
- net AM4:14: now also AM4.18 (Y13), S62.2 (VOUT); no longer AM5.17 (Y14), S79.2 (VOUT)
- net AM4:15: now also AM4.17 (Y14), S63.2 (VOUT); no longer AM5.16 (Y15), S80.2 (VOUT)
- net AM4:2: now also AM4.8 (Y1), S50.2 (VOUT); no longer AM5.7 (Y2), S67.2 (VOUT)
- net AM4:3: now also AM4.7 (Y2), S51.2 (VOUT); no longer AM5.6 (Y3), S68.2 (VOUT)
- net AM4:4: now also AM4.6 (Y3), S52.2 (VOUT); no longer AM5.5 (Y4), S69.2 (VOUT)
- net AM4:5: now also AM4.5 (Y4), S53.2 (VOUT); no longer AM5.4 (Y5), S70.2 (VOUT)
- net AM4:6: now also AM4.4 (Y5), S54.2 (VOUT); no longer AM5.3 (Y6), S71.2 (VOUT)
- net AM4:7: now also AM4.3 (Y6), S55.2 (VOUT); no longer AM5.2 (Y7), S72.2 (VOUT)
- net AM4:8: now also AM4.2 (Y7), S56.2 (VOUT); no longer AM5.23 (Y8), S73.2 (VOUT)
- net AM4:9: now also AM4.23 (Y8), S57.2 (VOUT); no longer AM5.22 (Y9), S74.2 (VOUT)
- net AM5: now also AM5.1 (Z), U1.6; no longer AM6.1 (Z), U1.7
- net AM5:1: no longer AM6.8 (Y1), S82.2 (VOUT)
- net AM5:10: now also AM5.22 (Y9), S74.2 (VOUT); no longer AM6.21 (Y10), S91.2 (VOUT)
- net AM5:11: now also AM5.21 (Y10), S75.2 (VOUT); no longer AM6.20 (Y11), S92.2 (VOUT)
- net AM5:12: now also AM5.20 (Y11), S76.2 (VOUT); no longer AM6.19 (Y12), S93.2 (VOUT)
- net AM5:13: now also AM5.19 (Y12), S77.2 (VOUT); no longer AM6.18 (Y13), S94.2 (VOUT)
- net AM5:14: now also AM5.18 (Y13), S78.2 (VOUT); no longer AM6.17 (Y14), S95.2 (VOUT)
- net AM5:15: now also AM5.17 (Y14), S79.2 (VOUT); no longer AM6.16 (Y15), S96.2 (VOUT)
- net AM5:2: now also AM5.8 (Y1), S66.2 (VOUT); no longer AM6.7 (Y2), S83.2 (VOUT)
- net AM5:3: now also AM5.7 (Y2), S67.2 (VOUT); no longer AM6.6 (Y3), S84.2 (VOUT)
- net AM5:4: now also AM5.6 (Y3), S68.2 (VOUT); no longer AM6.5 (Y4), S85.2 (VOUT)
- net AM5:5: now also AM5.5 (Y4), S69.2 (VOUT); no longer AM6.4 (Y5), S86.2 (VOUT)
- net AM5:6: now also AM5.4 (Y5), S70.2 (VOUT); no longer AM6.3 (Y6), S87.2 (VOUT)
- net AM5:7: now also AM5.3 (Y6), S71.2 (VOUT); no longer AM6.2 (Y7), S88.2 (VOUT)
- net AM5:8: now also AM5.2 (Y7), S72.2 (VOUT); no longer AM6.23 (Y8), S89.2 (VOUT)
- net AM5:9: now also AM5.23 (Y8), S73.2 (VOUT); no longer AM6.22 (Y9), S90.2 (VOUT)
- net CONTROL1: no longer AM1.11 (S1), AM2.11 (S1), AM3.11 (S1), AM4.11 (S1), AM5.11 (S1), AM6.11 (S1), U1.12
- net CONTROL2: now also AM1.11 (S2), AM2.11 (S2), AM3.11 (S2), AM4.11 (S2), AM5.11 (S2), AM6.11 (S2), U1.12; no longer AM1.14 (S2), AM2.14 (S2), AM3.14 (S2), AM4.14 (S2), AM5.14 (S2), AM6.14 (S2), U1.13
- net CONTROL3: now also AM1.14 (S3), AM2.14 (S3), AM3.14 (S3), AM4.14 (S3), AM5.14 (S3), AM6.14 (S3), U1.13; no longer AM1.13 (S3), AM2.13 (S3), AM3.13 (S3), AM4.13 (S3), AM5.13 (S3), AM6.13 (S3), U1.14
- net AM0:15 renamed AM1:16
- net AM5:0 renamed AM6:1
- new net AM2:16: AM2.16 (Y15), S32.2 (VOUT)
- new net AM3:16: AM3.16 (Y15), S48.2 (VOUT)
- new net AM4:16: AM4.16 (Y15), S64.2 (VOUT)
- new net AM5:16: AM5.16 (Y15), S80.2 (VOUT)
- new net AM6: AM6.1 (Z), U1.7
- new net AM6:10: AM6.22 (Y9), S90.2 (VOUT)
- new net AM6:11: AM6.21 (Y10), S91.2 (VOUT)
- new net AM6:12: AM6.20 (Y11), S92.2 (VOUT)
- new net AM6:13: AM6.19 (Y12), S93.2 (VOUT)
- new net AM6:14: AM6.18 (Y13), S94.2 (VOUT)
- new net AM6:15: AM6.17 (Y14), S95.2 (VOUT)
- new net AM6:16: AM6.16 (Y15), S96.2 (VOUT)
- new net AM6:2: AM6.8 (Y1), S82.2 (VOUT)
- new net AM6:3: AM6.7 (Y2), S83.2 (VOUT)
- new net AM6:4: AM6.6 (Y3), S84.2 (VOUT)
- new net AM6:5: AM6.5 (Y4), S85.2 (VOUT)
- new net AM6:6: AM6.4 (Y5), S86.2 (VOUT)
- new net AM6:7: AM6.3 (Y6), S87.2 (VOUT)
- new net AM6:8: AM6.2 (Y7), S88.2 (VOUT)
- new net AM6:9: AM6.23 (Y8), S89.2 (VOUT)
- new net CONTROL4: AM1.13 (S4), AM2.13 (S4), AM3.13 (S4), AM4.13 (S4), AM5.13 (S4), AM6.13 (S4), U1.14
