File: hardware/kicad/96_key/96_key.kicad_pcb (KiCad board)
At the start: 2 copper layers, 370.8 x 126.5 mm, 329 parts, among them U1 PM254-1-14-W-8.5

Commit message: Ok
Parts:
- removed the H0 at (208.8, 137.2)
- removed the REF** at (218.9, 234.5)
- added REF**: MountingHole_2.2mm_M2_Pad, MountingHole:MountingHole_2.2mm_M2_Pad, F.Cu at (219.0, 177.5)
- added REF**: MountingHole_2.2mm_M2_Pad, MountingHole:MountingHole_2.2mm_M2_Pad, F.Cu at (117.5, 177.5)
- added REF**: MountingHole_2.2mm_M2_Pad, MountingHole:MountingHole_2.2mm_M2_Pad, F.Cu at (320.5, 177.5)
- H0 (x26): value MountingHole_3.2mm_M3_Pad -> MountingHole_2.5mm_Pad; footprint MountingHole:MountingHole_3.2mm_M3_Pad -> MountingHole:MountingHole_2.5mm_Pad
- moved H0 14.0 mm to (354.9, 250.7)
- moved H0 14.0 mm to (385.3, 137.2)
- moved H0 14.0 mm to (72.9, 137.2)
- moved H0 14.0 mm to (42.4, 250.7)
- moved H0 10.0 mm to (87.0, 250.7)
- moved H0 10.0 mm to (117.5, 137.2)
- moved H0 10.0 mm to (340.7, 137.2)
- moved H0 10.0 mm to (310.2, 250.7)
- moved H0 6.00 mm to (265.6, 250.7)
- moved H0 6.00 mm to (162.1, 137.2)
- moved H0 6.00 mm to (296.1, 137.2)
- moved H0 6.00 mm to (131.7, 250.7)
- moved H0 2.00 mm to (251.4, 137.2)
- moved H0 2.00 mm to (176.3, 250.7)
- moved H0 2.00 mm to (220.9, 250.7)

Commit message: Ok
Other:
- board size 370.8 x 126.5 mm -> 352.8 x 125.8 mm
Changed lines of the file:
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@@
 		)
 	)
-	(gr_rect
-		(start 28.431096 131.1148)
-		(end 399.271096 257.6576)
+	(gr_poly
+		(pts
+			(xy 37.5 257.25) (xy 37.5 232) (xy 47.75 232) (xy 47.75 214.25) (xy 57.75 214.25) (xy 57.75 196)
+			(xy 47.75 196) (xy 47.75 179.25) (xy 57.75 179.25) (xy 57.75 161.25) (xy 68 161.25) (xy 68 131.5)
+			(xy 390.25 131.5) (xy 390.25 161) (xy 380 161) (xy 380 178.5) (xy 369.75 178.5) (xy 369.75 196.75)
+			(xy 380 196.75) (xy 380 213.75) (xy 369.75 213.75) (xy 369.75 231.25) (xy 359.75 231.25) (xy 359.75 257.25)
+		)
 		(stroke
 			(width 0.05)
-			(type default)
+			(type solid)
 		)
 		(fill no)

Commit message: Ok
Parts:
- REF** (x3): value MountingHole_2.2mm_M2_Pad -> MountingHole_2.5mm_Pad; footprint MountingHole:MountingHole_2.2mm_M2_Pad -> MountingHole:MountingHole_2.5mm_Pad
Changed lines of the file:
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@@
 		)
 	)
-	(footprint "MountingHole:MountingHole_2.2mm_M2_Pad"
+	(footprint "MountingHole:MountingHole_2.5mm_Pad"
 		(layer "F.Cu")
 		(at 219 177.5)
-		(descr "Mounting Hole 2.2mm, M2, generated by kicad-footprint-generator mountinghole.py")
-		(tags "mountinghole M2")
+		(descr "Mounting Hole 2.5mm, generated by kicad-footprint-generator mountinghole.py")
+		(tags "mountinghole")
 		(property "Reference" "REF**"
-			(at 0 -3.15 0)
+			(at 0 -3.45 0)
 			(layer "F.SilkS")
 			(effects
@@
 			)
 		)
-		(property "Value" "MountingHole_2.2mm_M2_Pad"
-			(at 0 3.15 0)
+		(property "Value" "MountingHole_2.5mm_Pad"
+			(at 0 3.45 0)
 			(layer "F.Fab")
 			(effects
@@
 		(fp_circle
 			(center 0 0)
-			(end 2.2 0)
+			(end 2.5 0)
 			(stroke
 				(width 0.15)
@@
 		(fp_circle
 			(center 0 0)
-			(end 2.45 0)
+			(end 2.75 0)
 			(stroke
 				(width 0.05)
@@
 		(pad "1" thru_hole circle
 			(at 0 0)
-			(size 4.4 4.4)
-			(drill 2.2)
+			(size 5 5)
+			(drill 2.5)
 			(layers "*.Cu" "*.Mask")
 			(remove_unused_layers no)
@@
 		)
 	)
-	(footprint "MountingHole:MountingHole_2.2mm_M2_Pad"
+	(footprint "MountingHole:MountingHole_2.5mm_Pad"
 		(layer "F.Cu")
 		(at 117.5 177.5)
-		(descr "Mounting Hole 2.2mm, M2, generated by kicad-footprint-generator mountinghole.py")
-		(tags "mountinghole M2")
+		(descr "Mounting Hole 2.5mm, generated by kicad-footprint-generator mountinghole.py")
+		(tags "mountinghole")
 		(property "Reference" "REF**"
-			(at 0 -3.15 0)
+			(at 0 -3.45 0)
 			(layer "F.SilkS")
 			(effects
@@
 			)
 		)
-		(property "Value" "MountingHole_2.2mm_M2_Pad"
-			(at 0 3.15 0)
+		(property "Value" "MountingHole_2.5mm_Pad"
+			(at 0 3.45 0)
 			(layer "F.Fab")
 			(effects
@@
 		(fp_circle
 			(center 0 0)
-			(end 2.2 0)
+			(end 2.5 0)
 			(stroke
 				(width 0.15)
@@
 		(fp_circle
 			(center 0 0)
-			(end 2.45 0)
+			(end 2.75 0)
 			(stroke
 				(width 0.05)
@@
 		(pad "1" thru_hole circle
 			(at 0 0)
-			(size 4.4 4.4)
-			(drill 2.2)
+			(size 5 5)
+			(drill 2.5)
 			(layers "*.Cu" "*.Mask")
 			(remove_unused_layers no)
@@
 		)
 	)
-	(footprint "MountingHole:MountingHole_2.2mm_M2_Pad"
+	(footprint "MountingHole:MountingHole_2.5mm_Pad"
 		(layer "F.Cu")
 		(at 320.5 177.5)
-		(descr "Mounting Hole 2.2mm, M2, generated by kicad-footprint-generator mountinghole.py")
-		(tags "mountinghole M2")
+		(descr "Mounting Hole 2.5mm, generated by kicad-footprint-generator mountinghole.py")
+		(tags "mountinghole")
 		(property "Reference" "REF**"
-			(at 0 -3.15 0)
+			(at 0 -3.45 0)
 			(layer "F.SilkS")
 			(effects
@@
 			)
 		)
-		(property "Value" "MountingHole_2.2mm_M2_Pad"
-			(at 0 3.15 0)
+		(property "Value" "MountingHole_2.5mm_Pad"
+			(at 0 3.45 0)
 			(layer "F.Fab")
 			(effects
@@
 		(fp_circle
 			(center 0 0)
-			(end 2.2 0)
+			(end 2.5 0)
 			(stroke
 				(width 0.15)
@@
 		(fp_circle
 			(center 0 0)
-			(end 2.45 0)
+			(end 2.75 0)
 			(stroke
 				(width 0.05)
@@
 		(pad "1" thru_hole circle
 			(at 0 0)
-			(size 4.4 4.4)
-			(drill 2.2)
+			(size 5 5)
+			(drill 2.5)
 			(layers "*.Cu" "*.Mask")
 			(remove_unused_layers no)

Commit message: Feedback https://www.reddit.com/r/KiCad/comments/1pkh416/review_request_192key_hall_effect_keyboard
Parts:
- moved H0 1.00 mm to (265.6, 251.7)
- moved H0 1.00 mm to (354.9, 251.7)
- moved H0 1.00 mm to (87.0, 251.7)
- moved H0 1.00 mm to (176.3, 251.7)
- moved H0 1.00 mm to (310.2, 251.7)
- moved H0 1.00 mm to (131.7, 251.7)
- moved H0 1.00 mm to (220.9, 251.7)
- moved H0 1.00 mm to (42.4, 251.7)
Routing:
- net +3.3V: track 319.0 -> 2311.7 mm, vias 102 -> 204
- net GND: track 25.4 -> 20.0 mm, vias 0 -> 16
- added copper zone on B.Cu, net +3.3V
- added copper zone on F.Cu, net GND
