File: hardware/kicad/96_key/96_key.kicad_pcb (KiCad board)
At the start: 2 copper layers, 352.8 x 125.8 mm, 330 parts, among them U1 PM254-1-14-W-8.5

Commit message: Ok
Routing:
- net AM1:7: track 69.1 -> 70.4 mm
- net AM5:15: track 70.2 -> 71.5 mm
- net AM2:15: track 70.2 -> 71.5 mm
- net AM0:8: track 71.0 -> 72.2 mm
- net AM3:8: track 71.0 -> 72.2 mm
- net AM4:0: track 72.5 -> 73.7 mm
- net AM1:0: track 72.5 -> 73.7 mm
- net AM2:8: track 71.0 -> 72.1 mm
- net AM3:15: track 70.2 -> 71.2 mm
- net AM0:15: track 70.2 -> 71.2 mm
- net AM1:6: track 49.5 -> 50.4 mm
- net AM4:7: track 69.1 -> 70.0 mm
- net AM2:14: track 50.6 -> 51.5 mm
- net AM5:14: track 50.6 -> 51.5 mm
- net AM3:9: track 51.3 -> 52.2 mm
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
Commit message: Ok
Parts:
- moved H0 7.00 mm to (251.4, 130.2)
- moved H0 7.00 mm to (162.1, 130.2)
- moved H0 7.00 mm to (117.5, 130.2)
- moved H0 7.00 mm to (385.3, 130.2)
- moved H0 7.00 mm to (340.7, 130.2)
- moved H0 7.00 mm to (296.1, 130.2)
- moved H0 7.00 mm to (72.9, 130.2)
- moved U1 5.90 mm to (213.8, 135.3)
Routing:
- net +3.3V: track 2311.7 -> 2368.9 mm
- net AM1: track 160.9 -> 169.8 mm
- net AM0: track 118.5 -> 125.8 mm
- net AM2: track 207.6 -> 214.2 mm
- net AM4: track 124.3 -> 130.4 mm
- net AM3: track 85.4 -> 91.4 mm
- net CONTROL3: track 383.6 -> 389.5 mm
- net CONTROL2: track 383.7 -> 389.1 mm
- net CONTROL1: track 378.6 -> 382.9 mm
- net AM5: track 176.9 -> 181.0 mm
- net CONTROL0: track 377.8 -> 381.2 mm
- net AM3:12: track 11.3 -> 12.0 mm
- net AM5:12: track 11.3 -> 12.0 mm
- net AM4:3: track 13.6 -> 14.2 mm
- net GND: vias 16 -> 17
Other:
- board size 352.8 x 125.8 mm -> 352.8 x 131.8 mm

Commit message: Ok
Parts:
- AM0, AM1, AM2, AM3, AM4, AM5: footprint jlcpcb:SSOP-24_L8.1-W5.3-P0.65-LS7.8-BL -> jlcpcb:TSSOP-24_L7.8-W4.4-P0.65-LS6.4-BL
