File: hardware/kicad/96_key/96_key.kicad_pcb (KiCad board)
At the start: 2 copper layers, 352.8 x 131.8 mm, 330 parts, among them U1 PM254-1-14-W-8.5

Commit message: Ok
Parts:
- H0: moved to F.Cu
- H1, H11, H13, H14, H15, H16, H17, H18, H19, H2, H20, H21, H22, H23, H24, H25, H26, H27, H28, H3, H4, H5, H6, H7, H9: renamed from H0; moved to F.Cu
- turned H0 to 0 degrees
- turned H1 to 0 degrees
- turned H11 to 0 degrees
- turned H13 to 0 degrees
- turned H14 to 0 degrees
- turned H15 to 0 degrees
- turned H16 to 0 degrees
- turned H17 to 0 degrees
- turned H18 to 0 degrees
- turned H19 to 0 degrees
- turned H2 to 0 degrees
- turned H20 to 0 degrees
- turned H21 to 0 degrees
- turned H22 to 0 degrees
- turned H23 to 0 degrees
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- renumbered REF** to H10, REF** to H12, REF** to H8
Routing:
- net CONTROL0: track 381.2 -> 384.0 mm
- net AM2: track 214.2 -> 215.4 mm
- net CONTROL3: track 389.5 -> 388.4 mm
- net CONTROL1: track 382.9 -> 383.8 mm
- net AM0: track 125.8 -> 126.6 mm
- net AM1: track 169.8 -> 170.4 mm
- net GND: track 20.4 -> 21.1 mm
- net CONTROL2: track 389.1 -> 389.6 mm
Other:
- board text added: "https://github.com/DumpsterDoofus/keyboard_accordion/tree/2cf37cad98c52a38ec58199ef9a22818f4d123ae/hardware/kicad/96_key"

Commit message: Ok
Parts:
- AM1: renamed from AM0; value CD74HC4067SM96 -> 74HC4067PW,118
- AM2: renamed from AM1; value CD74HC4067SM96 -> 74HC4067PW,118
- AM3: renamed from AM2; value CD74HC4067SM96 -> 74HC4067PW,118
- AM4: renamed from AM3; value CD74HC4067SM96 -> 74HC4067PW,118
- AM5: renamed from AM4; value CD74HC4067SM96 -> 74HC4067PW,118
- AM6: renamed from AM5; value CD74HC4067SM96 -> 74HC4067PW,118
- renumbered C0 to C1, C9 to C10, C195 to C100, C196 to C101, C197 to C102, C10 to C11, C11 to C12, C12 to C13, C13 to C14, C14 to C15, C15 to C16, C16 to C17, C17 to C18, C18 to C19, C1 to C2, C19 to C20, C20 to C21, C21 to C22, C22 to C23, C23 to C24, C24 to C25, C25 to C26, C26 to C27, C27 to C28, C28 to C29, C2 to C3, C29 to C30, C30 to C31, C31 to C32, C32 to C33, C33 to C34, C34 to C35, C35 to C36, C36 to C37, C37 to C38, C38 to C39, C3 to C4, C39 to C40, C40 to C41, C41 to C42, C42 to C43, C43 to C44, C44 to C45, C45 to C46, C46 to C47, C47 to C48, C48 to C49, C4 to C5, C49 to C50, C50 to C51, C51 to C52, C52 to C53, C53 to C54, C54 to C55, C55 to C56, C56 to C57, C57 to C58, C58 to C59, C5 to C6, C59 to C60, C60 to C61, C61 to C62, C62 to C63, C63 to C64, C64 to C65, C65 to C66, C66 to C67, C67 to C68, C68 to C69, C6 to C7, C69 to C70, C70 to C71, C71 to C72, C72 to C73, C73 to C74, C74 to C75, C75 to C76, C76 to C77, C77 to C78, C78 to C79, C7 to C8, C79 to C80, C80 to C81, C81 to C82, C82 to C83, C83 to C84, C84 to C85, C85 to C86, C86 to C87, C87 to C88, C88 to C89, C8 to C9, C89 to C90, C90 to C91, C91 to C92, C92 to C93, C93 to C94, C94 to C95, C95 to C96, C192 to C97, C193 to C98, C194 to C99, H0 to H1, H9 to H10, H10 to H11, H11 to H12, H12 to H13, H13 to H14, H14 to H15, H15 to H16, H16 to H17, H17 to H18, H18 to H19, H1 to H2, H19 to H20, H20 to H21, H21 to H22, H22 to H23, H23 to H24, H24 to H25, H25 to H26, H26 to H27, H27 to H28, H28 to H29, H2 to H3, H3 to H4, H4 to H5, H5 to H6, H6 to H7, H7 to H8, H8 to H9, KEY0 to KEY1, KEY9 to KEY10, KEY10 to KEY11, KEY11 to KEY12, KEY12 to KEY13, KEY13 to KEY14, KEY14 to KEY15, KEY15 to KEY16, KEY16 to KEY17, KEY17 to KEY18, KEY18 to KEY19, KEY1 to KEY2, KEY19 to KEY20, KEY20 to KEY21, KEY21 to KEY22, KEY22 to KEY23, KEY23 to KEY24, KEY24 to KEY25, KEY25 to KEY26, KEY26 to KEY27, KEY27 to KEY28, KEY28 to KEY29, KEY2 to KEY3, KEY29 to KEY30, KEY30 to KEY31, KEY31 to KEY32, KEY32 to KEY33, KEY33 to KEY34, KEY34 to KEY35, KEY35 to KEY36, KEY36 to KEY37, KEY37 to KEY38, KEY38 to KEY39, KEY3 to KEY4, KEY39 to KEY40, KEY40 to KEY41, KEY41 to KEY42, KEY42 to KEY43, KEY43 to KEY44, KEY44 to KEY45, KEY45 to KEY46, KEY46 to KEY47, KEY47 to KEY48, KEY48 to KEY49, KEY4 to KEY5, KEY49 to KEY50, KEY50 to KEY51, KEY51 to KEY52, KEY52 to KEY53, KEY53 to KEY54, KEY54 to KEY55, KEY55 to KEY56, KEY56 to KEY57, KEY57 to KEY58, KEY58 to KEY59, KEY5 to KEY6, KEY59 to KEY60, KEY60 to KEY61, KEY61 to KEY62, KEY62 to KEY63, KEY63 to KEY64, KEY64 to KEY65, KEY65 to KEY66, KEY66 to KEY67, KEY67 to KEY68, KEY68 to KEY69, KEY6 to KEY7, KEY69 to KEY70, KEY70 to KEY71, KEY71 to KEY72, KEY72 to KEY73, KEY73 to KEY74, KEY74 to KEY75, KEY75 to KEY76, KEY76 to KEY77, KEY77 to KEY78, KEY78 to KEY79, KEY7 to KEY8, KEY79 to KEY80, KEY80 to KEY81, KEY81 to KEY82, KEY82 to KEY83, KEY83 to KEY84, KEY84 to KEY85, KEY85 to KEY86, KEY86 to KEY87, KEY87 to KEY88, KEY88 to KEY89, KEY8 to KEY9, KEY89 to KEY90, KEY90 to KEY91, KEY91 to KEY92, KEY92 to KEY93, KEY93 to KEY94, KEY94 to KEY95, KEY95 to KEY96, S0 to S1, S9 to S10, S10 to S11, S11 to S12, S12 to S13, S13 to S14, S14 to S15, S15 to S16, S16 to S17, S17 to S18, S18 to S19, S1 to S2, S19 to S20, S20 to S21, S21 to S22, S22 to S23, S23 to S24, S24 to S25, S25 to S26, S26 to S27, S27 to S28, S28 to S29, S2 to S3, S29 to S30, S30 to S31, S31 to S32, S32 to S33, S33 to S34, S34 to S35, S35 to S36, S36 to S37, S37 to S38, S38 to S39, S3 to S4, S39 to S40, S40 to S41, S41 to S42, S42 to S43, S43 to S44, S44 to S45, S45 to S46, S46 to S47, S47 to S48, S48 to S49, S4 to S5, S49 to S50, S50 to S51, S51 to S52, S52 to S53, S53 to S54, S54 to S55, S55 to S56, S56 to S57, S57 to S58, S58 to S59, S5 to S6, S59 to S60, S60 to S61, S61 to S62, S62 to S63, S63 to S64, S64 to S65, S65 to S66, S66 to S67, S67 to S68, S68 to S69, S6 to S7, S69 to S70, S70 to S71, S71 to S72, S72 to S73, S73 to S74, S74 to S75, S75 to S76, S76 to S77, S77 to S78, S78 to S79, S7 to S8, S79 to S80, S80 to S81, S81 to S82, S82 to S83, S83 to S84, S84 to S85, S85 to S86, S86 to S87, S87 to S88, S88 to S89, S8 to S9, S89 to S90, S90 to S91, S91 to S92, S92 to S93, S93 to S94, S94 to S95, S95 to S96
Connections:
- net AM0:15 renamed AM1:16
- net AM5:0 renamed AM6:1
- AM1 pad 1: AM0 -> AM1
- AM1 pad 10: CONTROL0 -> CONTROL1
- AM1 pad 11: CONTROL1 -> CONTROL2
- AM1 pad 13: CONTROL3 -> CONTROL4
- AM1 pad 14: CONTROL2 -> CONTROL3
- AM1 pad 17: AM0:14 -> AM1:15
- AM1 pad 18: AM0:13 -> AM1:14
- AM1 pad 19: AM0:12 -> AM1:13
- AM1 pad 2: AM0:7 -> AM1:8
- AM1 pad 20: AM0:11 -> AM1:12
- AM1 pad 21: AM0:10 -> AM1:11
- AM1 pad 22: AM0:9 -> AM1:10
- AM1 pad 23: AM0:8 -> AM1:9
- AM1 pad 3: AM0:6 -> AM1:7
- AM1 pad 4: AM0:5 -> AM1:6
- AM1 pad 5: AM0:4 -> AM1:5
- AM1 pad 6: AM0:3 -> AM1:4
- AM1 pad 7: AM0:2 -> AM1:3
- AM1 pad 8: AM0:1 -> AM1:2
- AM1 pad 9: AM0:0 -> AM1:1
- AM2 pad 1: AM1 -> AM2
- AM2 pad 10: CONTROL0 -> CONTROL1
- AM2 pad 11: CONTROL1 -> CONTROL2
- AM2 pad 13: CONTROL3 -> CONTROL4
- AM2 pad 14: CONTROL2 -> CONTROL3
- AM2 pad 16: AM1:15 -> AM2:16
- AM2 pad 17: AM1:14 -> AM2:15
- AM2 pad 18: AM1:13 -> AM2:14
- AM2 pad 19: AM1:12 -> AM2:13
- AM2 pad 2: AM1:7 -> AM2:8
- AM2 pad 20: AM1:11 -> AM2:12
- AM2 pad 21: AM1:10 -> AM2:11
- AM2 pad 22: AM1:9 -> AM2:10
- AM2 pad 23: AM1:8 -> AM2:9
- AM2 pad 3: AM1:6 -> AM2:7
- AM2 pad 4: AM1:5 -> AM2:6
- AM2 pad 5: AM1:4 -> AM2:5
- AM2 pad 6: AM1:3 -> AM2:4
- AM2 pad 7: AM1:2 -> AM2:3
- AM2 pad 8: AM1:1 -> AM2:2
- AM2 pad 9: AM1:0 -> AM2:1
- AM3 pad 1: AM2 -> AM3
- AM3 pad 10: CONTROL0 -> CONTROL1
- AM3 pad 11: CONTROL1 -> CONTROL2
- AM3 pad 13: CONTROL3 -> CONTROL4
- AM3 pad 14: CONTROL2 -> CONTROL3
- AM3 pad 16: AM2:15 -> AM3:16
- AM3 pad 17: AM2:14 -> AM3:15
- AM3 pad 18: AM2:13 -> AM3:14
- AM3 pad 19: AM2:12 -> AM3:13
- AM3 pad 2: AM2:7 -> AM3:8
- AM3 pad 20: AM2:11 -> AM3:12
- AM3 pad 21: AM2:10 -> AM3:11
- AM3 pad 22: AM2:9 -> AM3:10
- AM3 pad 23: AM2:8 -> AM3:9
- AM3 pad 3: AM2:6 -> AM3:7
- AM3 pad 4: AM2:5 -> AM3:6
- AM3 pad 5: AM2:4 -> AM3:5
- AM3 pad 6: AM2:3 -> AM3:4
- AM3 pad 7: AM2:2 -> AM3:3
- AM3 pad 8: AM2:1 -> AM3:2
- AM3 pad 9: AM2:0 -> AM3:1
- AM4 pad 1: AM3 -> AM4
- AM4 pad 10: CONTROL0 -> CONTROL1
- AM4 pad 11: CONTROL1 -> CONTROL2
- AM4 pad 13: CONTROL3 -> CONTROL4
- AM4 pad 14: CONTROL2 -> CONTROL3
- AM4 pad 16: AM3:15 -> AM4:16
- AM4 pad 17: AM3:14 -> AM4:15
- AM4 pad 18: AM3:13 -> AM4:14
- AM4 pad 19: AM3:12 -> AM4:13
- AM4 pad 2: AM3:7 -> AM4:8
- AM4 pad 20: AM3:11 -> AM4:12
- AM4 pad 21: AM3:10 -> AM4:11
- AM4 pad 22: AM3:9 -> AM4:10
- AM4 pad 23: AM3:8 -> AM4:9
- AM4 pad 3: AM3:6 -> AM4:7
- AM4 pad 4: AM3:5 -> AM4:6
- AM4 pad 5: AM3:4 -> AM4:5
- AM4 pad 6: AM3:3 -> AM4:4
- AM4 pad 7: AM3:2 -> AM4:3
- AM4 pad 8: AM3:1 -> AM4:2
- AM4 pad 9: AM3:0 -> AM4:1
- AM5 pad 1: AM4 -> AM5
- AM5 pad 10: CONTROL0 -> CONTROL1
- AM5 pad 11: CONTROL1 -> CONTROL2
- AM5 pad 13: CONTROL3 -> CONTROL4
- AM5 pad 14: CONTROL2 -> CONTROL3
- AM5 pad 16: AM4:15 -> AM5:16
- AM5 pad 17: AM4:14 -> AM5:15
- AM5 pad 18: AM4:13 -> AM5:14
- AM5 pad 19: AM4:12 -> AM5:13
- AM5 pad 2: AM4:7 -> AM5:8
- AM5 pad 20: AM4:11 -> AM5:12
- AM5 pad 21: AM4:10 -> AM5:11
- AM5 pad 22: AM4:9 -> AM5:10
- AM5 pad 23: AM4:8 -> AM5:9
- AM5 pad 3: AM4:6 -> AM5:7
- AM5 pad 4: AM4:5 -> AM5:6
- AM5 pad 5: AM4:4 -> AM5:5
- AM5 pad 6: AM4:3 -> AM5:4
- AM5 pad 7: AM4:2 -> AM5:3
- AM5 pad 8: AM4:1 -> AM5:2
- AM5 pad 9: AM4:0 -> AM5:1
- AM6 pad 1: AM5 -> AM6
- AM6 pad 10: CONTROL0 -> CONTROL1
- AM6 pad 11: CONTROL1 -> CONTROL2
- AM6 pad 13: CONTROL3 -> CONTROL4
- AM6 pad 14: CONTROL2 -> CONTROL3
- AM6 pad 16: AM5:15 -> AM6:16
- AM6 pad 17: AM5:14 -> AM6:15
- AM6 pad 18: AM5:13 -> AM6:14
- AM6 pad 19: AM5:12 -> AM6:13
- AM6 pad 2: AM5:7 -> AM6:8
- AM6 pad 20: AM5:11 -> AM6:12
- AM6 pad 21: AM5:10 -> AM6:11
- AM6 pad 22: AM5:9 -> AM6:10
- AM6 pad 23: AM5:8 -> AM6:9
- AM6 pad 3: AM5:6 -> AM6:7
- AM6 pad 4: AM5:5 -> AM6:6
- AM6 pad 5: AM5:4 -> AM6:5
- AM6 pad 6: AM5:3 -> AM6:4
- AM6 pad 7: AM5:2 -> AM6:3
- AM6 pad 8: AM5:1 -> AM6:2
- S1 pad 2: AM0:0 -> AM1:1
- S10 pad 2: AM0:9 -> AM1:10
- S11 pad 2: AM0:10 -> AM1:11
- S12 pad 2: AM0:11 -> AM1:12
- S13 pad 2: AM0:12 -> AM1:13
- S14 pad 2: AM0:13 -> AM1:14
- S15 pad 2: AM0:14 -> AM1:15
- S17 pad 2: AM1:0 -> AM2:1
- S18 pad 2: AM1:1 -> AM2:2
- S19 pad 2: AM1:2 -> AM2:3
- S2 pad 2: AM0:1 -> AM1:2
- S20 pad 2: AM1:3 -> AM2:4
- S21 pad 2: AM1:4 -> AM2:5
- S22 pad 2: AM1:5 -> AM2:6
- S23 pad 2: AM1:6 -> AM2:7
- S24 pad 2: AM1:7 -> AM2:8
- S25 pad 2: AM1:8 -> AM2:9
- S26 pad 2: AM1:9 -> AM2:10
- S27 pad 2: AM1:10 -> AM2:11
- S28 pad 2: AM1:11 -> AM2:12
- S29 pad 2: AM1:12 -> AM2:13
- S3 pad 2: AM0:2 -> AM1:3
- S30 pad 2: AM1:13 -> AM2:14
- S31 pad 2: AM1:14 -> AM2:15
- S32 pad 2: AM1:15 -> AM2:16
- S33 pad 2: AM2:0 -> AM3:1
- S34 pad 2: AM2:1 -> AM3:2
- S35 pad 2: AM2:2 -> AM3:3
- S36 pad 2: AM2:3 -> AM3:4
- S37 pad 2: AM2:4 -> AM3:5
- S38 pad 2: AM2:5 -> AM3:6
- S39 pad 2: AM2:6 -> AM3:7
- S4 pad 2: AM0:3 -> AM1:4
- S40 pad 2: AM2:7 -> AM3:8
- S41 pad 2: AM2:8 -> AM3:9
- S42 pad 2: AM2:9 -> AM3:10
- S43 pad 2: AM2:10 -> AM3:11
- S44 pad 2: AM2:11 -> AM3:12
- S45 pad 2: AM2:12 -> AM3:13
- S46 pad 2: AM2:13 -> AM3:14
- S47 pad 2: AM2:14 -> AM3:15
- S48 pad 2: AM2:15 -> AM3:16
- S49 pad 2: AM3:0 -> AM4:1
- S5 pad 2: AM0:4 -> AM1:5
- S50 pad 2: AM3:1 -> AM4:2
- S51 pad 2: AM3:2 -> AM4:3
- S52 pad 2: AM3:3 -> AM4:4
- S53 pad 2: AM3:4 -> AM4:5
- S54 pad 2: AM3:5 -> AM4:6
- S55 pad 2: AM3:6 -> AM4:7
- S56 pad 2: AM3:7 -> AM4:8
- S57 pad 2: AM3:8 -> AM4:9
- S58 pad 2: AM3:9 -> AM4:10
- S59 pad 2: AM3:10 -> AM4:11
- S6 pad 2: AM0:5 -> AM1:6
- S60 pad 2: AM3:11 -> AM4:12
- S61 pad 2: AM3:12 -> AM4:13
- S62 pad 2: AM3:13 -> AM4:14
- S63 pad 2: AM3:14 -> AM4:15
- S64 pad 2: AM3:15 -> AM4:16
- S65 pad 2: AM4:0 -> AM5:1
- S66 pad 2: AM4:1 -> AM5:2
- S67 pad 2: AM4:2 -> AM5:3
- S68 pad 2: AM4:3 -> AM5:4
- S69 pad 2: AM4:4 -> AM5:5
- S7 pad 2: AM0:6 -> AM1:7
- S70 pad 2: AM4:5 -> AM5:6
- S71 pad 2: AM4:6 -> AM5:7
- S72 pad 2: AM4:7 -> AM5:8
- S73 pad 2: AM4:8 -> AM5:9
- S74 pad 2: AM4:9 -> AM5:10
- S75 pad 2: AM4:10 -> AM5:11
- S76 pad 2: AM4:11 -> AM5:12
- S77 pad 2: AM4:12 -> AM5:13
- S78 pad 2: AM4:13 -> AM5:14
- S79 pad 2: AM4:14 -> AM5:15
- S8 pad 2: AM0:7 -> AM1:8
- S80 pad 2: AM4:15 -> AM5:16
- S82 pad 2: AM5:1 -> AM6:2
- S83 pad 2: AM5:2 -> AM6:3
- S84 pad 2: AM5:3 -> AM6:4
- S85 pad 2: AM5:4 -> AM6:5
- S86 pad 2: AM5:5 -> AM6:6
- S87 pad 2: AM5:6 -> AM6:7
- S88 pad 2: AM5:7 -> AM6:8
- S89 pad 2: AM5:8 -> AM6:9
- S9 pad 2: AM0:8 -> AM1:9
- S90 pad 2: AM5:9 -> AM6:10
- S91 pad 2: AM5:10 -> AM6:11
- S92 pad 2: AM5:11 -> AM6:12
- S93 pad 2: AM5:12 -> AM6:13
- S94 pad 2: AM5:13 -> AM6:14
- S95 pad 2: AM5:14 -> AM6:15
- S96 pad 2: AM5:15 -> AM6:16
- U1 pad 10: AM0 -> AM1
- U1 pad 11: CONTROL0 -> CONTROL1
- U1 pad 12: CONTROL1 -> CONTROL2
- U1 pad 13: CONTROL2 -> CONTROL3
- U1 pad 14: CONTROL3 -> CONTROL4
- U1 pad 5: AM3 -> AM4
- U1 pad 6: AM4 -> AM5
- U1 pad 7: AM5 -> AM6
- U1 pad 8: AM2 -> AM3
- U1 pad 9: AM1 -> AM2
Routing:
- net CONTROL4: track 0.00 -> 388.4 mm, vias 0 -> 9
- net CONTROL0: track 384.0 -> 0.00 mm, vias 9 -> 0
- net AM6: track 0.00 -> 181.5 mm, vias 0 -> 2
- net AM0: track 126.6 -> 0.00 mm, vias 2 -> 0
- net AM3: track 91.6 -> 215.4 mm
- net AM0:0: track 83.1 -> 0.00 mm
- net AM3:0: track 83.1 -> 0.00 mm
- net AM2:0: track 83.1 -> 0.00 mm
- net AM2:16: track 0.00 -> 81.3 mm
- net AM5:16: track 0.00 -> 81.3 mm
- net AM4:0: track 73.7 -> 0.00 mm
- net AM1:0: track 73.5 -> 0.00 mm
- net AM0:8: track 72.2 -> 0.00 mm
- net AM6:9: track 0.00 -> 71.7 mm
- net AM6:16: track 0.00 -> 71.5 mm
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
Commit message: Ok
Other:
- board text added: "https://github.com/DumpsterDoofus/keyboard_accordion/releases/tag/0.2.0"
- board text removed: "https://github.com/DumpsterDoofus/keyboard_accordion/tree/2cf37cad98c52a38ec58199ef9a22818f4d123ae/hardware/kicad/96_key"
Changed lines of the file:
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@@
 		(layer "Edge.Cuts")
 	)
-	(gr_text "https://github.com/DumpsterDoofus/keyboard_accordion/tree/2cf37cad98c52a38ec58199ef9a22818f4d123ae/hardware/kicad/96_key"
-		(at 127.95 232.2 0)
+	(gr_text "https://github.com/DumpsterDoofus/keyboard_accordion/releases/tag/0.2.0"
+		(at 165.45 128.95 0)
 		(layer "F.SilkS")
 		(effects
