File: hardware/kicad/daughterboard/daughterboard.kicad_pcb (KiCad board)
At the start: 2 copper layers, 71.1 x 40.6 mm, 8 parts, among them J1 X6511FV-24-C85D32, J2 X6511FV-24-C85D32, U1 XDJK-0051-025, U2 BX-PM2.54-1-14PY, U3 BX-PM2.54-1-14PY

Commit message: Ok
Parts:
- added REF1: MountingHole_2.5mm_Pad, MountingHole:MountingHole_2.5mm_Pad, F.Cu at (96.5, 19.5)
- added REF2: MountingHole_2.5mm_Pad, MountingHole:MountingHole_2.5mm_Pad, F.Cu at (65.2, 46.5)
- added REF3: MountingHole_2.5mm_Pad, MountingHole:MountingHole_2.5mm_Pad, F.Cu at (127.8, 46.5)

Commit message: Ok
Parts:
- moved R2 13.9 mm to (120.6, 39.6), turned to 90 degrees
Routing:
- net GND: track 44.4 -> 3.40 mm
- net +3.3V: track 37.0 -> 65.8 mm
- net Net-(J2-35_TX8): track 4.35 -> 8.02 mm
- net AM4: vias 1 -> 0
- net AM3: vias 1 -> 0
- net AM5: vias 1 -> 0
- net AM2: vias 1 -> 0
- net AM1: vias 1 -> 0
- net AM0: vias 1 -> 0
- added copper zone on F.Cu, net GND
- removed copper zone on F.Cu, net +3.3V

Commit message: Ok
Parts:
- renumbered REF1 to H1, REF2 to H2, REF3 to H3
Routing:
- net GND: track 3.40 -> 0.86 mm
Other:
- board text added: "Left board"
- board text added: "Right board"
- board text added: "Teensy 4.1"
Changed lines of the file:
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@@
 			(crossoutdnponfab yes)
 			(subtractmaskfromsilk no)
-			(outputformat 1)
+			(outputformat 4)
 			(mirror no)
-			(drillshape 1)
+			(drillshape 0)
 			(scaleselection 1)
-			(outputdirectory "")
+			(outputdirectory "/home/peter/Pictures/")
 		)
 	)
@@
 		(at 88.1228 38.4556 180)
 		(property "Reference" "C1"
-			(at 0 -4 0)
+			(at -3.9272 0.0056 0)
 			(layer "F.SilkS")
 			(effects
@@
 		(at 70.6701 40.5763)
 		(property "Reference" "U1"
-			(at 0 -6.35 0)
+			(at 0 -7.7763 0)
 			(layer "F.SilkS")
 			(effects
@@
 		(at 88.0804 40.7924 180)
 		(property "Reference" "R1"
-			(at 0 -4 0)
+			(at -4.0196 0.0924 0)
 			(layer "F.SilkS")
 			(effects
@@
 		(at 120.6 39.6 90)
 		(property "Reference" "R2"
-			(at 0 -4 90)
+			(at -0.25 2.55 90)
 			(layer "F.SilkS")
 			(effects
@@
 		(at 100.7364 43.4848)
 		(property "Reference" "U2"
-			(at 0 -4 0)
+			(at -19.6364 0.0652 0)
 			(layer "F.SilkS")
 			(effects
@@
 		(descr "Mounting Hole 2.5mm, generated by kicad-footprint-generator mountinghole.py")
 		(tags "mountinghole")
-		(property "Reference" "REF2"
-			(at 0 -3.45 0)
+		(property "Reference" "H2"
+			(at 3.95 0.1 0)
 			(layer "F.SilkS")
 			(effects
@@
 		(descr "Mounting Hole 2.5mm, generated by kicad-footprint-generator mountinghole.py")
 		(tags "mountinghole")
-		(property "Reference" "REF1"
-			(at 0 -3.45 0)
+		(property "Reference" "H1"
+			(at 4.5 -0.1 0)
 			(layer "F.SilkS")
 			(effects
@@
 		(at 96.4184 30.1244)
 		(property "Reference" "J2"
-			(at 0 -4 0)
+			(at -32.1184 0.1756 0)
 			(layer "F.SilkS")
 			(effects
@@
 		(descr "Mounting Hole 2.5mm, generated by kicad-footprint-generator mountinghole.py")
 		(tags "mountinghole")
-		(property "Reference" "REF3"
-			(at 0 -3.45 0)
+		(property "Reference" "H3"
+			(at -4.15 0.1 0)
 			(layer "F.SilkS")
 			(effects
@@
 		(at 96.4184 14.8844)
 		(property "Reference" "J1"
-			(at 0 -4 0)
+			(at -31.8684 0.0156 0)
 			(layer "F.SilkS")
 			(effects
@@
 		(at 100.7364 35.8648)
 		(property "Reference" "U3"
-			(at 0 -4 0)
+			(at -19.5364 -0.1648 0)
 			(layer "F.SilkS")
 			(effects
@@
 		(layer "Edge.Cuts")
 	)
+	(gr_text "Right board"
+		(at 94.6 47 0)
+		(layer "F.SilkS")
+		(effects
+			(font
+				(size 1.397 1.397)
+				(thickness 0.2794)
+				(bold yes)
+			)
+			(justify left bottom)
+		)
+	)
+	(gr_text "Left board"
+		(at 95.6 34 0)
+		(layer "F.SilkS")
+		(effects
+			(font
+				(size 1.397 1.397)
+				(thickness 0.2794)
+				(bold yes)
+			)
+			(justify left bottom)
+		)
+	)
+	(gr_text "Teensy 4.1"
+		(at 91.8 24 0)
+		(layer "F.SilkS")
+		(effects
+			(font
+				(size 1.397 1.397)
+				(thickness 0.2794)
+				(bold yes)
+			)
+			(justify left bottom)
+		)
+	)
 	(segment
 		(start 86.6004 43.3188)
@@
 		(net 2)
 	)
-	(segment
-		(start 91.8464 35.8648)
-		(end 89.3064 35.8648)
-		(width 1.524)
-		(layer "B.Cu")
-		(net 2)
-	)

Commit message: Ok
Other:
- board text added: "https://github.com/DumpsterDoofus/keyboard_accordion/releases/tag/0.2.0"
Changed lines of the file:
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@@
 		(layer "Edge.Cuts")
 	)
-	(gr_text "Right board"
-		(at 94.6 47 0)
+	(gr_text "Left board"
+		(at 95.4 46.8 0)
 		(layer "F.SilkS")
 		(effects
@@
 		)
 	)
-	(gr_text "Left board"
-		(at 95.6 34 0)
+	(gr_text "https://github.com/DumpsterDoofus/keyboard_accordion/releases/tag/0.2.0"
+		(at 67.2 12.6 0)
 		(layer "F.SilkS")
 		(effects
+			(font
+				(size 1 1)
+				(thickness 0.2)
+				(bold yes)
+			)
+			(justify left bottom)
+		)
+	)
+	(gr_text "Right board"
+		(at 94.6 33.8 0)
+		(layer "F.SilkS")
+		(effects

Commit message: Ok
Parts:
- moved R1 11.7 mm to (76.5, 41.7), turned to 90 degrees
- moved C1 9.82 mm to (79.0, 42.0), turned to 90 degrees
- turned R2 to -90 degrees
Connections:
- J2 pad 10: AM6 -> AM7
- J2 pad 11: AM7 -> AM8
- J2 pad 12: AM8 -> AM9
- J2 pad 13: AM9 -> AM10
- J2 pad 16: AM10 -> AM11
- J2 pad 17: AM11 -> AM12
- J2 pad 18: CONTROL0 -> CONTROL1
- J2 pad 19: CONTROL1 -> CONTROL2
- J2 pad 20: CONTROL2 -> CONTROL3
- J2 pad 21: CONTROL3 -> CONTROL4
- J2 pad 4: AM0 -> AM1
- J2 pad 5: AM1 -> AM2
- J2 pad 6: AM2 -> AM3
- J2 pad 7: AM3 -> AM4
- J2 pad 8: AM4 -> AM5
- J2 pad 9: AM5 -> AM6
- R2 pad 1: +3.3V -> Net-(J2-35_TX8)
- R2 pad 2: Net-(J2-35_TX8) -> +3.3V
- U2 pad 10: AM5 -> AM6
- U2 pad 11: CONTROL0 -> CONTROL1
- U2 pad 12: CONTROL1 -> CONTROL2
- U2 pad 13: CONTROL2 -> CONTROL3
- U2 pad 14: CONTROL3 -> CONTROL4
- U2 pad 5: AM0 -> AM1
- U2 pad 6: AM1 -> AM2
- U2 pad 7: AM2 -> AM3
- U2 pad 8: AM3 -> AM4
- U2 pad 9: AM4 -> AM5
- U3 pad 10: AM11 -> AM12
- U3 pad 11: CONTROL0 -> CONTROL1
- U3 pad 12: CONTROL1 -> CONTROL2
- U3 pad 13: CONTROL2 -> CONTROL3
- U3 pad 14: CONTROL3 -> CONTROL4
- U3 pad 5: AM6 -> AM7
- U3 pad 6: AM7 -> AM8
- U3 pad 7: AM8 -> AM9
- U3 pad 8: AM9 -> AM10
- U3 pad 9: AM10 -> AM11
Routing:
- net AM6: track 7.53 -> 38.5 mm
- net AM0: track 27.9 -> 0.00 mm
- net CONTROL4: track 0.00 -> 13.7 mm
- net CONTROL0: track 13.7 -> 0.00 mm
- net AM12: track 0.00 -> 6.06 mm
- net AM5: track 38.6 -> 36.0 mm
- net AM4: track 35.5 -> 33.0 mm
- net AM10: track 6.06 -> 7.53 mm
- net AM3: track 32.2 -> 31.1 mm
