File: hardware/pcb/3_key_v2/3_key_v2.kicad_sch (KiCad schematic)
At the start: 55 parts, among them J1 USB TYPE-C-31-M-12, J2 JST SWD debug header, SW1 Pushbutton, SW2 Pushbutton, U1 AP7361C-Y5-13, U2 ME6211A33M3G-N, U3 TLV74311PDBVR, U4 RP2354A, Y1 ABM8-272-T3

Commit message: Ok
Parts:
- removed ADC1, ADC2: TLA2528IRTER, jlcpcb:WQFN-16_L3.0-W3.0-P0.50-TL-EP1.7, symbol jlcpcb:TLA2528IRTER
- removed AM1, AM2: CD4052BMT/TR, jlcpcb:TSSOP-16_L5.0-W4.4-P0.65-LS6.4-BL, symbol jlcpcb:CD4052BMT_TR
- added ADC1, ADC2: TLA2518IRTET, jlcpcb:WQFN-16_L3.0-W3.0-P0.50-TL-EP1.7, symbol jlcpcb:TLA2518IRTET
- added AM1, AM2: CD4052BLQ/TR, jlcpcb:VQFN-16_L3.0-W3.0-P0.50-BL-EP1.4, symbol jlcpcb:CD4052BLQ_TR
Connections:
- net +3.3V: now also ADC1.10 (DVDD), ADC2.10 (DVDD)
- net +4V: now also ADC1.7 (AVDD), ADC2.7 (AVDD), AM1.16 (VDD), AM2.16 (VDD)
- net AM1:1: now also ADC1.2 (AIN3/GPIO3), AM1.3 (COMY)
- net AM1:2: now also ADC1.1 (AIN2/GPIO2), AM1.13 (COMX)
- net AM2:1: now also ADC2.1 (AIN2/GPIO2), AM2.3 (COMY)
- net AM2:2: now also ADC2.2 (AIN3/GPIO3), AM2.13 (COMX)
- net CONTROL_A: now also AM1.10 (A), AM2.10 (A)
- net CONTROL_B: now also AM1.9 (B), AM2.9 (B)
- net GND: now also ADC1.15 (AIN0/GPIO0), ADC1.16 (AIN1/GPIO1), ADC1.3 (AIN4/GPIO4), ADC1.4 (AIN5/GPIO5), ADC1.5 (AIN6/GPIO6), ADC1.6 (AIN7/GPIO7), ADC1.9 (GND), ADC2.15 (AIN0/GPIO0), ADC2.16 (AIN1/GPIO1), ADC2.17 (EP), ADC2.3 (AIN4/GPIO4), ADC2.4 (AIN5/GPIO5), ADC2.5 (AIN6/GPIO6), ADC2.6 (AIN7/GPIO7), ADC2.9 (GND), AM1.11 (X3), AM1.12 (X0), AM1.14 (X1), AM1.15 (X2), AM1.17 (EP), AM1.2 (Y2), AM1.4 (Y3), AM1.5 (Y1), AM1.6 (INH), AM1.7 (VEE), AM1.8 (VSS), AM2.11 (X3), AM2.12 (X0), AM2.14 (X1), AM2.15 (X2), AM2.17 (EP), AM2.2 (Y2), AM2.4 (Y3), AM2.5 (Y1), AM2.6 (INH), AM2.7 (VEE), AM2.8 (VSS)
- net at S2.2 (VOUT): now also AM2.1 (Y0)
- net at C8.1: now also ADC2.8 (DECAP)
- net at C5.1: now also ADC1.8 (DECAP)
- net at S1.2 (VOUT): now also AM1.1 (Y0)
- net MISO2: now reaches U4.12 (GPIO8)
- net MISO2: now also ADC2.12 (SDO)
- net CS2: now reaches U4.13 (GPIO9)
- net CS2: now also ADC2.11 (~{CS})
- net SCLK2: now reaches U4.14 (GPIO10)
- net SCLK2: now also ADC2.13 (SCLK)
- net MOSI2: now reaches U4.15 (GPIO11)
- net MOSI2: now also ADC2.14 (SDI)
- net SCL1 renamed CS1
- net CS1: now also ADC1.11 (~{CS})
- net SCL2 renamed MOSI1
- net MOSI1: now also ADC1.14 (SDI)
- net SDA1 renamed MISO1
- net MISO1: now also ADC1.12 (SDO)
- net SDA2 renamed SCLK1
- net SCLK1: now also ADC1.13 (SCLK)
- no-connect marks 36 -> 29
